File: myrio_pcb.kicad_pcb (KiCad board)
At the start: 4 copper layers, 191.1 x 89.5 mm, 136 parts, among them J1 DB9, P1 CONN_02X17, P2 CONN_02X17, Q1 PN2222A, Q10 PN2222A, Q11 PN2222A, Q12 PN2222A, Q13 PN2222A, Q14 PN2222A, Q15 PN2222A, Q16 PN2222A, Q17 PN2222A, Q18 PN2222A, Q19 PN2222A, Q2 PN2222A, Q20 PN2222A, Q21 PN2222A, Q3 PN2222A, Q4 PN2222A, Q5 PN2222A, Q6 PN2222A, Q7 PN2222A, Q8 PN2222A, Q9 PN2222A, U1 stacked-DB9, U10 INA219, U11 INA219, U13 INA219, U14 stacked-rj45-LED, U15 stacked-rj45-LED, U16 12V regulator, U2 stacked-DB9, U3 stacked-rj45-LED, U4 stacked-rj45-LED, U5 stacked-rj45-LED, U6 BNO055, U7 stacked-rj45-LED, U9 LM1084IT-5.0/NOPB

Commit message: the schematic looks good just have to add the screw terminals and ethernet footprints. I also edited the pcb file so that it has some helpful test on the left and right side
Other:
- board text added: "a0 a1 4 digital i2c lines"
- board text added: "cap gnd move next to motor gnd screw terminals"
- board text added: "power- battery connection and converters battery+ bat- 4 connectors for 24V booster 4 connectors for 5V booster"
Changed lines of the file:
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@@
-(kicad_pcb (version 4) (host pcbnew 4.0.6)
+(kicad_pcb (version 4) (host pcbnew 4.0.3-stable)
   (general
     (links 409)
@@
     (area 8.481287 0.983 228.500715 113.698001)
     (thickness 1.6)
-    (drawings 84)
+    (drawings 87)
     (tracks 1552)
     (zones 0)
@@
     )
   )
+  (gr_text "a0\na1\n4 digital i2c lines" (at -7.366 57.15) (layer F.Cu)
+    (effects (font (size 1.5 1.5) (thickness 0.3)))
+  )
+  (gr_text "cap gnd move next to motor gnd screw terminals" (at 245.872 100.076) (layer F.Cu)
+    (effects (font (size 1.5 1.5) (thickness 0.3)))
+  )
+  (gr_text "power- battery connection and converters\nbattery+\nbat-\n4 connectors for 24V booster\n4 connectors for 5V booster\n\n" (at 246.634 70.104) (layer F.Cu)
+    (effects (font (size 1.5 1.5) (thickness 0.3)))
+  )
   (gr_text gnd (at 183.8706 99.30384) (layer F.SilkS)
