File: myrio_pcb.kicad_pcb (KiCad board)
At the start: 4 copper layers, 191.1 x 89.5 mm, 136 parts, among them J1 DB9, P1 CONN_02X17, P2 CONN_02X17, Q1 PN2222A, Q10 PN2222A, Q11 PN2222A, Q12 PN2222A, Q13 PN2222A, Q14 PN2222A, Q15 PN2222A, Q16 PN2222A, Q17 PN2222A, Q18 PN2222A, Q19 PN2222A, Q2 PN2222A, Q20 PN2222A, Q21 PN2222A, Q3 PN2222A, Q4 PN2222A, Q5 PN2222A, Q6 PN2222A, Q7 PN2222A, Q8 PN2222A, Q9 PN2222A, U1 stacked-DB9, U10 INA219, U11 INA219, U13 INA219, U14 stacked-rj45-LED, U15 stacked-rj45-LED, U16 12V regulator, U2 stacked-DB9, U3 stacked-rj45-LED, U4 stacked-rj45-LED, U5 stacked-rj45-LED, U6 BNO055, U7 stacked-rj45-LED, U9 LM1084IT-5.0/NOPB

Commit message: donezo
Parts:
- removed C1, C2, C3, C4: CP1, Capacitors_THT:CP_Radial_Tantal_D4.5mm_P2.50mm
- removed D23: D, Diodes_THT:D_DO-35_SOD27_P5.08mm_Vertical_AnodeUp
- removed J1: DB9, Connectors:DB9FD
- removed Q21: PN2222A, footprints:pn2222
- removed R21: 100K, Resistors_THT:R_Axial_DIN0204_L3.6mm_D1.6mm_P5.08mm_Horizontal
- removed R31: R, Resistors_THT:R_Axial_DIN0204_L3.6mm_D1.6mm_P5.08mm_Horizontal
- removed RE21: relay, footprints:relay
- removed REF** (x4): 1pin, Connectors:1pin
- removed U16: 12V regulator, TO_SOT_Packages_THT:TO-220_Vertical
- removed U9: LM1084IT-5.0/NOPB, TO_SOT_Packages_THT:TO-220_Vertical
- added S11: 2pinscrew, footprints:screwinconnector++, F.Cu at (219.7, 102.2)
- added U8: stacked-DB9, footprints:DB9-doublestacked_PR, F.Cu at (208.5, 33.5)
- H1: footprint footprints:bmp180_ref -> footprints:bmp180
- Q1, Q10, Q11, Q12, Q13, Q14, Q15, Q16, Q17, Q18, Q19, Q2, Q20, Q3, Q4, Q5, Q6, Q7, Q8, Q9: footprint footprints:pn2222 -> TO_SOT_Packages_THT:TO-92_Inline_Narrow_Oval
- S1, S10, S2, S3, S4, S5, S6, S7, S8, S9: footprint footprints:screwinconnector -> footprints:screwinconnector++
- U14, U15, U3, U4, U5, U7: footprint footprints:stacked-rj45_Final -> footprints:stacked-rj45_Final++
- moved S10 204.9 mm to (226.7, 93.3)
- moved S9 204.8 mm to (226.7, 81.9)
- moved S8 204.7 mm to (226.7, 70.5)
- moved S5 185.4 mm to (23.5, 62.2), turned to 270 degrees
- moved S4 184.9 mm to (23.5, 50.8)
- moved S2 183.6 mm to (23.5, 73.7)
- moved S1 20.5 mm to (226.7, 59.1), turned to 90 degrees
- moved S6 17.9 mm to (189.2, 102.2), turned to 0 degrees
- moved D21 9.53 mm to (158.8, 100.3)
- moved U1 7.63 mm to (154.3, 39.0)
- moved U2 7.63 mm to (188.0, 39.0)
- moved U15 6.99 mm to (132.1, 30.5)
- moved U14 5.71 mm to (112.4, 30.5)
- moved D22 5.12 mm to (200.0, 97.2), turned to 0 degrees
- moved U7 4.44 mm to (92.7, 30.5)
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Connections:
- 220ohm1 pad 2: friction_gnd -> DGND
- 220ohm2 pad 2: friction_gnd -> DGND
- 220ohm3 pad 2: friction_gnd -> DGND
- 220ohm4 pad 2: friction_gnd -> DGND
- P1 pad 1: Net-(P1-Pad1) -> (no net)
- P1 pad 10: Net-(P1-Pad10) -> (no net)
- P1 pad 12: friction_gnd -> DGND
- P1 pad 14: Net-(P1-Pad14) -> (no net)
- P1 pad 16: friction_gnd -> DGND
- P1 pad 2: Net-(P1-Pad2) -> (no net)
- P1 pad 20: friction_gnd -> DGND
- P1 pad 24: friction_gnd -> DGND
- P1 pad 28: friction_gnd -> DGND
- P1 pad 30: friction_gnd -> DGND
- P1 pad 33: Net-(P1-Pad33) -> (no net)
- P1 pad 4: Net-(P1-Pad4) -> (no net)
- P1 pad 6: friction_gnd -> DGND
- P1 pad 8: friction_gnd -> DGND
- P2 pad 1: Net-(P2-Pad1) -> (no net)
- P2 pad 10: Net-(P2-Pad10) -> (no net)
- P2 pad 14: Net-(P2-Pad14) -> (no net)
- P2 pad 2: Net-(P2-Pad2) -> (no net)
- P2 pad 33: Net-(P2-Pad33) -> (no net)
- P2 pad 4: Net-(P2-Pad4) -> (no net)
- P2 pad 6: friction_gnd -> DGND
- P2 pad 7: Net-(P2-Pad7) -> (no net)
- P2 pad 9: Net-(P2-Pad9) -> (no net)
- Q1 pad 1: friction_gnd -> DGND
- Q10 pad 1: friction_gnd -> DGND
- Q11 pad 1: friction_gnd -> DGND
- Q12 pad 1: friction_gnd -> DGND
- Q13 pad 1: friction_gnd -> DGND
- Q14 pad 1: friction_gnd -> DGND
- Q15 pad 1: friction_gnd -> DGND
- Q16 pad 1: friction_gnd -> DGND
- Q17 pad 1: friction_gnd -> DGND
- Q18 pad 1: friction_gnd -> DGND
- Q19 pad 1: friction_gnd -> DGND
- Q2 pad 1: friction_gnd -> DGND
- Q20 pad 1: friction_gnd -> DGND
- Q3 pad 1: friction_gnd -> DGND
- Q4 pad 1: friction_gnd -> DGND
- Q5 pad 1: friction_gnd -> DGND
- Q6 pad 1: friction_gnd -> DGND
- Q7 pad 1: friction_gnd -> DGND
- Q8 pad 1: friction_gnd -> DGND
- Q9 pad 1: friction_gnd -> DGND
- RE1 pad 5: Net-(RE1-Pad5) -> (no net)
- RE10 pad 5: Net-(RE10-Pad5) -> (no net)
- RE11 pad 5: Net-(RE11-Pad5) -> (no net)
- RE12 pad 5: Net-(RE12-Pad5) -> (no net)
- RE13 pad 6: Net-(RE13-Pad6) -> (no net)
- RE15 pad 6: Net-(RE15-Pad6) -> (no net)
- RE18 pad 10: Net-(RE18-Pad10) -> (no net)
- RE19 pad 1: friction_gnd -> DGND
- RE2 pad 5: Net-(RE2-Pad5) -> (no net)
- RE20 pad 1: friction_gnd -> DGND
- RE3 pad 5: Net-(RE3-Pad5) -> (no net)
- RE4 pad 5: Net-(RE4-Pad5) -> (no net)
- RE5 pad 1: Net-(RE5-Pad1) -> (no net)
- RE9 pad 5: Net-(RE9-Pad5) -> (no net)
- S1 pad 1: VCC_IN -> batt_in
- S1 pad 2: friction_gnd -> DGND
- S10 pad 1: 5V -> 12V
- S10 pad 2: friction_gnd -> DGND
- S6 pad 2: friction_gnd -> DGND
- S7 pad 1: motor_pwr -> 24V
- S7 pad 2: friction_gnd -> 24V
- S8 pad 1: VCC_IN -> 12V
- S8 pad 2: friction_gnd -> DGND
- S9 pad 1: 12V -> 24V
- S9 pad 2: friction_gnd -> DGND
- U1 pad 14: friction_gnd -> DGND
- U1 pad 15: friction_gnd -> DGND
- U1 pad 16: friction_gnd -> DGND
- U1 pad 17: friction_gnd -> DGND
- U1 pad 18: friction_gnd -> DGND
- U1 pad 5: friction_gnd -> DGND
- U1 pad 6: friction_gnd -> DGND
- U1 pad 7: friction_gnd -> DGND
- U1 pad 8: friction_gnd -> DGND
- U1 pad 9: friction_gnd -> DGND
- U10 pad 5: Net-(U10-Pad5) -> (no net)
- U10 pad 6: Net-(U10-Pad6) -> (no net)
- U11 pad 5: Net-(U11-Pad5) -> (no net)
- U11 pad 6: Net-(U11-Pad6) -> (no net)
- U11 pad 7: 24V -> 12V
- U11 pad 8: VCC_IN -> batt_in
- U13 pad 5: Net-(U13-Pad5) -> (no net)
- U13 pad 6: Net-(U13-Pad6) -> (no net)
- U14 pad 14: Net-(U14-Pad14) -> (no net)
- U14 pad 17: Net-(U14-Pad17) -> (no net)
- U14 pad 18: Net-(U14-Pad18) -> (no net)
- U14 pad 19: Net-(U14-Pad19) -> (no net)
- U14 pad 20: Net-(U14-Pad20) -> (no net)
- U14 pad 21: Net-(U14-Pad21) -> (no net)
- U14 pad 22: Net-(U14-Pad22) -> (no net)
- U14 pad 23: Net-(U14-Pad23) -> (no net)
- U14 pad 24: Net-(U14-Pad24) -> (no net)
- U14 pad 6: Net-(U14-Pad6) -> (no net)
- U14 pad 8: Net-(U14-Pad8) -> (no net)
- U15 pad 12: Net-(U15-Pad12) -> (no net)
- U15 pad 13: Net-(U15-Pad13) -> (no net)
- U15 pad 15: Net-(U15-Pad15) -> (no net)
- U15 pad 16: Net-(U15-Pad16) -> (no net)
- U15 pad 17: Net-(U15-Pad17) -> (no net)
- U15 pad 18: Net-(U15-Pad18) -> (no net)
- U15 pad 19: Net-(U15-Pad19) -> (no net)
- U15 pad 20: Net-(U15-Pad20) -> (no net)
- U15 pad 21: Net-(U15-Pad21) -> (no net)
- U15 pad 22: Net-(U15-Pad22) -> (no net)
- U15 pad 23: Net-(U15-Pad23) -> (no net)
- U15 pad 24: Net-(U15-Pad24) -> (no net)
- U2 pad 14: friction_gnd -> DGND
- U2 pad 15: friction_gnd -> DGND
- U2 pad 16: friction_gnd -> DGND
- U2 pad 17: friction_gnd -> DGND
- U2 pad 18: friction_gnd -> DGND
- U2 pad 5: friction_gnd -> DGND
- U2 pad 6: friction_gnd -> DGND
- U2 pad 7: friction_gnd -> DGND
- U2 pad 8: friction_gnd -> DGND
- U2 pad 9: friction_gnd -> DGND
- U3 pad 17: Net-(U3-Pad17) -> (no net)
- U3 pad 18: Net-(U3-Pad18) -> (no net)
- U3 pad 19: Net-(U3-Pad19) -> (no net)
- U3 pad 20: Net-(U3-Pad20) -> (no net)
- U3 pad 21: Net-(U3-Pad21) -> (no net)
- U3 pad 22: Net-(U3-Pad22) -> (no net)
- U3 pad 23: Net-(U3-Pad23) -> (no net)
- U3 pad 24: Net-(U3-Pad24) -> (no net)
- U4 pad 17: Net-(U4-Pad17) -> (no net)
- U4 pad 18: Net-(U4-Pad18) -> (no net)
- U4 pad 19: Net-(U4-Pad19) -> (no net)
- U4 pad 20: Net-(U4-Pad20) -> (no net)
- U4 pad 21: Net-(U4-Pad21) -> (no net)
- U4 pad 22: Net-(U4-Pad22) -> (no net)
- U4 pad 23: Net-(U4-Pad23) -> (no net)
- U4 pad 24: Net-(U4-Pad24) -> (no net)
- U5 pad 17: Net-(U5-Pad17) -> (no net)
- U5 pad 18: Net-(U5-Pad18) -> (no net)
- U5 pad 19: Net-(U5-Pad19) -> (no net)
- U5 pad 20: Net-(U5-Pad20) -> (no net)
- U5 pad 21: Net-(U5-Pad21) -> (no net)
- U5 pad 22: Net-(U5-Pad22) -> (no net)
- U5 pad 23: Net-(U5-Pad23) -> (no net)
- U5 pad 24: Net-(U5-Pad24) -> (no net)
- U6 pad 10: Net-(U6-Pad10) -> (no net)
- U6 pad 2: Net-(U6-Pad2) -> (no net)
- U6 pad 6: Net-(U6-Pad6) -> (no net)
- U6 pad 7: Net-(U6-Pad7) -> (no net)
- U6 pad 8: Net-(U6-Pad8) -> (no net)
- U6 pad 9: Net-(U6-Pad9) -> (no net)
- U7 pad 14: Net-(U7-Pad14) -> (no net)
- U7 pad 16: Net-(U7-Pad16) -> (no net)
- U7 pad 17: Net-(U7-Pad17) -> (no net)
- U7 pad 18: Net-(U7-Pad18) -> (no net)
- U7 pad 19: Net-(U7-Pad19) -> (no net)
- U7 pad 20: Net-(U7-Pad20) -> (no net)
- U7 pad 21: Net-(U7-Pad21) -> (no net)
- U7 pad 22: Net-(U7-Pad22) -> (no net)
- U7 pad 23: Net-(U7-Pad23) -> (no net)
- U7 pad 24: Net-(U7-Pad24) -> (no net)
- U7 pad 4: Net-(U7-Pad4) -> (no net)
- U7 pad 5: Net-(U7-Pad5) -> (no net)
- U7 pad 6: Net-(U7-Pad6) -> (no net)
- U7 pad 7: Net-(U7-Pad7) -> (no net)
- U7 pad 8: Net-(U7-Pad8) -> (no net)
Routing:
- net VCC_IN: track 252.3 -> 0.00 mm, vias 8 -> 0
- net friction_gnd: track 195.1 -> 0.00 mm, vias 5 -> 0
- net A0: track 203.5 -> 53.5 mm, vias 1 -> 2
- net A1: track 197.0 -> 53.5 mm
- net motor_pwr: track 96.0 -> 0.00 mm, vias 2 -> 0
- net 24V: track 86.6 -> 0.00 mm, vias 3 -> 0
- net i2c_scl_2: track 179.6 -> 97.0 mm, vias 5 -> 4
- net motor_ctrl: track 55.7 -> 138.2 mm, vias 5 -> 2
- net batt_in: track 0.00 -> 73.9 mm, vias 0 -> 2
- net i2c_sda_2: track 167.9 -> 97.5 mm, vias 5 -> 2
- net non_critical_sda: track 341.1 -> 383.8 mm, vias 10 -> 13
- net DGND: track 0.00 -> 36.2 mm, vias 0 -> 1
- net 12V: track 168.4 -> 133.6 mm, vias 5 -> 2
- net i2c_sda_3: track 116.0 -> 144.7 mm, vias 3 -> 2
- net non_critical_scl: track 323.2 -> 350.2 mm
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- added copper zone on B.Cu, net 24V
- removed copper zone on F.Cu, net 24V
- removed copper zone on B.Cu, net friction_gnd
Other:
- board size 191.1 x 89.5 mm -> 212 x 89.5 mm
- board text added: "SCL2"
- board text added: "SCL3"
- board text added: "SDA2"
- board text added: "SDA3"
- board text removed: "Dgnd"
- board text removed: "Motor"
- board text removed: "Regulator"
