File: myrio_pcb.sch (KiCad schematic (older format))
At the start: 132 parts, among them J1 DB9, P1 CONN_02X17, P2 CONN_02X17, Q1 PN2222A, Q10 PN2222A, Q11 PN2222A, Q12 PN2222A, Q13 PN2222A, Q14 PN2222A, Q15 PN2222A, Q16 PN2222A, Q17 PN2222A, Q18 PN2222A, Q19 PN2222A, Q2 PN2222A, Q20 PN2222A, Q21 PN2222A, Q3 PN2222A, Q4 PN2222A, Q5 PN2222A, Q6 PN2222A, Q7 PN2222A, Q8 PN2222A, Q9 PN2222A, U1 stacked-DB9, U10 INA219, U11 INA219, U13 INA219, U14 stacked-rj45-LED, U15 stacked-rj45-LED, U16 12V regulator, U2 stacked-DB9, U3 stacked-rj45-LED, U4 stacked-rj45-LED, U5 stacked-rj45-LED, U6 BNO055, U7 stacked-rj45-LED, U9 LM1084IT-5.0/NOPB

Commit message: the schematic looks good just have to add the screw terminals and ethernet footprints. I also edited the pcb file so that it has some helpful test on the left and right side
Parts:
- removed C1, C2, C3, C4: CP1, Capacitors_THT:CP_Radial_Tantal_D4.5mm_P2.50mm, symbol CP1
- removed D23: D, Diodes_THT:D_DO-35_SOD27_P5.08mm_Vertical_AnodeUp, symbol D
- removed J1: DB9, Connectors:DB9FD, symbol DB9
- removed Q21: PN2222A, TO_SOT_Packages_THT:TO-92_Inline_Narrow_Oval, symbol PN2222A
- removed R21: 100K, Resistors_THT:R_Axial_DIN0204_L3.6mm_D1.6mm_P5.08mm_Horizontal, symbol R
- removed R31: R, Resistors_THT:R_Axial_DIN0204_L3.6mm_D1.6mm_P5.08mm_Horizontal, symbol R
- removed RE21: relay, footprints:relay, symbol relay
- removed S10, S7, S8, S9: 2pinscrew, footprints:screwinconnector, symbol 2pinscrew
- removed U16: 12V regulator, TO_SOT_Packages_THT:TO-220_Vertical, symbol LM1084IT-5.0/NOPB
- removed U9: LM1084IT-5.0/NOPB, TO_SOT_Packages_THT:TO-220_Vertical, symbol LM1084IT-5.0/NOPB
- added S? (x5): 2pinscrew, footprints:screwinconnector, symbol 2pinscrew
- added U?: stacked-DB9, footprints:DB9-doublestacked_PR, symbol stacked-DB9
Connections:
- net DGND is gone; now on net GND: D21.2 (A), H1.2 (gnd), P2.12 (P12), P2.16 (P16), P2.20 (P20), P2.24 (P24), P2.28 (P28), P2.30 (P30), P2.8 (P8), RE1.10 (NO), RE10.10 (NO), RE11.10 (NO), RE12.10 (NO), RE17.10 (NO), RE2.10 (NO), RE3.10 (NO), RE4.10 (NO), RE9.10 (NO), S3.2 (pin2), U10.2 (Gnd), U11.2 (Gnd), U13.2 (Gnd), U14.11, U14.16, U14.3, U14.7, U15.6, U3.10, U3.13, U3.2, U3.5, U4.10, U4.13, U4.2, U4.5, U5.10, U5.13, U5.2, U5.5, U6.3 (gnd), U7.10, U7.13, U7.2
- net 12V: now also U11.7 (VIN-)
- net 5V: now also S?.1 (pin1)
- net GND: now also S?.2 (pin2), S?.2 (pin2), S?.2 (pin2), S?.2 (pin2), U?.12, U?.9
- net VCC: now also S?.1 (pin1), S?.1 (pin1), S?.2 (pin2), U?.11, U?.5; no longer U11.7 (VIN-)
- net motor_ctrl: now also U?.10
- net VCC_IN renamed batt_in
- net batt_in: now also S?.1 (pin1), S?.1 (pin1)
- no-connect marks 108 -> 113
Other:
- note added: "Ripcord 24V pins"
- note added: "Voltage Converter Inputs"
- note removed: "Debugging Screw Terminals"

Commit message: cleaned schematic a bit and messed around the 12V battery signal have run a drc and annotate everything checks out
Parts:
- gave numbers to parts that had none: 6
Connections:
- net 12V: now also S10.1 (pin1), S8.1 (pin1)
- net batt_in: no longer S10.1 (pin1), S8.1 (pin1)
Other:
- note added: "Debugging"
- note added: "Power Supply Aliasing"
- note added: "Screw Terminals"
- note added: "Sense PWR toggle"
- note removed: "Power Supply"
- note removed: "just power and ground for the extra actuator"
- note removed: "non tof power toggle"
- note removed: "two pressure sensors will go into a screw terminal too ethernet board"
- moved on the sheet: S1, S2, S3, S4, S5, S6, U8
