File: myrio/myrio_pcb.sch (KiCad schematic (older format))
At the start: 122 parts, among them P1 CONN_02X17, P2 CONN_02X17, Q1 PN2222A, Q10 PN2222A, Q11 PN2222A, Q12 PN2222A, Q13 PN2222A, Q14 PN2222A, Q15 PN2222A, Q16 PN2222A, Q17 PN2222A, Q18 PN2222A, Q19 PN2222A, Q2 PN2222A, Q20 PN2222A, Q3 PN2222A, Q4 PN2222A, Q5 PN2222A, Q6 PN2222A, Q7 PN2222A, Q8 PN2222A, Q9 PN2222A, U1 stacked-DB9, U10 INA219, U11 INA219, U13 INA219, U14 stacked-rj45-LED, U15 stacked-rj45-LED, U2 stacked-DB9, U3 stacked-rj45-LED, U4 stacked-rj45-LED, U5 stacked-rj45-LED, U6 BNO055, U7 stacked-rj45-LED, U8 stacked-DB9

Commit message: moved the readme over here
Parts:
- added J1, J2, J3, J4: CONN_02X03, Pin_Headers:Pin_Header_Straight_2x03_Pitch2.54mm, symbol CONN_02X03
- S1, S10, S11, S2, S3, S4, S5, S6, S7, S8, S9: footprint footprints:screwinconnector -> footprints:screwinconnector++
- U14, U15, U3, U4, U5, U7: footprint footprints:stacked-rj45_Final -> footprints:stacked-rj45_Final++
Connections:
- net 5V: now also S11.2 (pin2); no longer S11.1 (pin1)
- net GND: now also S11.1 (pin1), S9.1 (pin1), U8.5; no longer S11.2 (pin2), S9.2 (pin2), U8.9
- net VCC: now also S9.2 (pin2), U8.9; no longer S7.2 (pin2), S9.1 (pin1), U8.5
- net critical_scl: now also J1.6 (P6), J3.6 (P6); no longer U4.3, U5.3
- net critical_sda: now also J2.6 (P6), J4.6 (P6); no longer U4.6, U5.6
- net i2c_scl_2: now also J1.2 (P2), J3.2 (P2)
- net i2c_sda_2: now also J2.2 (P2), J4.2 (P2)
- net magnetic_pwr: now also S7.2 (pin2)
- net non_critical_scl: now also J1.1 (P1), J3.1 (P1); no longer U4.11, U4.15, U4.7, U5.11, U5.15, U5.7
- net non_critical_sda: now also J2.1 (P1), J4.1 (P1); no longer U4.14, U4.16, U4.8, U5.14, U5.16, U5.8
- new net stress_scl: J3.3 (P3), J3.4 (P4), U5.11, U5.15, U5.3, U5.7
- new net stress_sda: J4.3 (P3), J4.4 (P4), U5.14, U5.16, U5.6, U5.8
- new net tof_scl: J1.3 (P3), J1.4 (P4), U4.11, U4.15, U4.3, U4.7
- new net tof_sda: J2.3 (P3), J2.4 (P4), U4.14, U4.16, U4.6, U4.8
- no-connect marks 113 -> 117

Commit message: flipped the 2ways functionality
Connections:
- net 2way_close_1: now also RE6.1 (NC); no longer RE6.10 (NO)
- net 2way_close_2: now also RE7.1 (NC); no longer RE7.10 (NO)
- net 2way_close_3: now also RE8.1 (NC); no longer RE8.10 (NO)
- net 2way_open_1: now also RE6.10 (NO); no longer RE6.1 (NC)
- net 2way_open_2: now also RE7.10 (NO); no longer RE7.1 (NC)
- net 2way_open_3: now also RE8.10 (NO); no longer RE8.1 (NC)
Changed lines of the file:
@@
 Text GLabel 14650 6050 2    30   Input ~ 0
 5V
+Text GLabel 14650 6350 2    30   Input ~ 0
+2way_close_1
 Text GLabel 14650 6200 2    30   Input ~ 0
-2way_close_1
-Text GLabel 14650 6350 2    30   Input ~ 0
 2way_open_1
 Text GLabel 13700 6200 0    30   Input ~ 0
@@
 Text GLabel 14650 6700 2    30   Input ~ 0
 5V
+Text GLabel 14650 7000 2    30   Input ~ 0
+2way_close_2
 Text GLabel 14650 6850 2    30   Input ~ 0
-2way_close_2
-Text GLabel 14650 7000 2    30   Input ~ 0
 2way_open_2
 Text GLabel 13700 6850 0    30   Input ~ 0
@@
 Text GLabel 14650 7350 2    30   Input ~ 0
 5V
+Text GLabel 14650 7650 2    30   Input ~ 0
+2way_close_3
 Text GLabel 14650 7500 2    30   Input ~ 0
-2way_close_3
-Text GLabel 14650 7650 2    30   Input ~ 0
 2way_open_3
 Text GLabel 13700 7500 0    30   Input ~ 0
@@
 	2250 6900 2250 7000
 Wire Wire Line
-	1050 7300 2250 7300
+	1050 7300 1450 7300
+Wire Wire Line
+	1450 7300 1700 7300
+Wire Wire Line
+	1700 7300 1850 7300
+Wire Wire Line
+	1850 7300 2250 7300
 Connection ~ 1450 7300
 Connection ~ 1850 7300
@@
 	5050 12300 5050 9250
 Wire Wire Line
-	10650 5650 10650 5750
+	10650 5650 10650 5700
+Wire Wire Line
+	10650 5700 10650 5750
 Wire Wire Line
 	10650 5700 10750 5700
@@
 	10550 5350 10650 5350
 Wire Wire Line
-	6650 5700 8500 5700
+	6650 5700 6750 5700
+Wire Wire Line
+	6750 5700 7000 5700
+Wire Wire Line
+	7000 5700 7250 5700
+Wire Wire Line
+	7250 5700 7500 5700
+Wire Wire Line
+	7500 5700 7750 5700
+Wire Wire Line
+	7750 5700 8000 5700
+Wire Wire Line
+	8000 5700 8250 5700
+Wire Wire Line
+	8250 5700 8500 5700
 Connection ~ 6750 5700
 Connection ~ 7000 5700
@@
 A1
 Wire Wire Line
-	22550 2150 22550 1450
+	22550 2150 22550 1800
+Wire Wire Line
+	22550 1800 22550 1450
 Wire Wire Line
 	22550 1800 23050 1800
@@
 	7350 1500 7350 1550
 Wire Wire Line
-	8000 1400 8000 1550
+	8000 1400 8000 1500
+Wire Wire Line
+	8000 1500 8000 1550
 $Comp
 L PWR_FLAG #FLG045

Commit message: added the router screw terminal
Parts:
- removed S7: 2pinscrew, footprints:screwinconnector++, symbol 2pinscrew
- added S?: 2pinscrew, footprints:screwinconnector++, symbol 2pinscrew
Connections:
- net 12V: now also S?.1 (pin1)
- net GND: now also S?.2 (pin2)
Other:
- note removed: "Ripcord 24V pins"

Commit message: undid changes writing stuff in the README
Parts:
- removed S?: 2pinscrew, footprints:screwinconnector++, symbol 2pinscrew
- added S7: 2pinscrew, footprints:screwinconnector++, symbol 2pinscrew
Connections:
- net 2way_close_1: now also RE6.10 (NO); no longer RE6.1 (NC)
- net 2way_close_2: now also RE7.10 (NO); no longer RE7.1 (NC)
- net 2way_close_3: now also RE8.10 (NO); no longer RE8.1 (NC)
- net 2way_open_1: now also RE6.1 (NC); no longer RE6.10 (NO)
- net 2way_open_2: now also RE7.1 (NC); no longer RE7.10 (NO)
- net 2way_open_3: now also RE8.1 (NC); no longer RE8.10 (NO)
- net VCC: now also S7.1 (pin1)
- net magnetic_pwr: now also S7.2 (pin2)
Other:
- note added: "Ripcord 24V pins"
