File: myrio/myrio_pcb.sch (KiCad schematic (older format))
At the start: 128 parts, among them J1 CONN_02X03, J2 CONN_02X03, J3 CONN_02X03, J4 CONN_02X03, P1 CONN_02X17, P2 CONN_02X17, Q1 PN2222A, Q10 PN2222A, Q11 PN2222A, Q12 PN2222A, Q13 PN2222A, Q14 PN2222A, Q15 PN2222A, Q16 PN2222A, Q17 PN2222A, Q18 PN2222A, Q19 PN2222A, Q2 PN2222A, Q20 PN2222A, Q3 PN2222A, Q4 PN2222A, Q5 PN2222A, Q6 PN2222A, Q7 PN2222A, Q8 PN2222A, Q9 PN2222A, T1 Phoenix_Contact_1935187, T2 Phoenix_Contact_1935187, T3 Phoenix_Contact_1935187, T4 Phoenix_Contact_1935187, U1 stacked-DB9, U10 INA219, U11 INA219, U13 INA219, U14 stacked-rj45-LED, U15 stacked-rj45-LED, U2 stacked-DB9, U3 stacked-rj45-LED, U4 stacked-rj45-LED, U5 stacked-rj45-LED, U6 BNO055, U7 stacked-rj45-LED, U8 stacked-DB9

Commit message: considering capacitors
Parts:
- added C1, C2, C3, C4, C5, C6, C7, C8, C9: C, Capacitors_THT:CP_Radial_D5.0mm_P2.50mm, symbol C
Connections:
- wire segments 209 -> 215
Changed lines of the file:
@@
 L PWR_FLAG #FLG019
 U 1 1 58EB21F4
-P 7050 1300
-F 0 "#FLG019" H 7050 1375 50  0001 C CNN
-F 1 "PWR_FLAG" H 7050 1450 50  0000 C CNN
-F 2 "" H 7050 1300 50  0001 C CNN
-F 3 "" H 7050 1300 50  0001 C CNN
-	1    7050 1300
+P 7050 1200
+F 0 "#FLG019" H 7050 1275 50  0001 C CNN
+F 1 "PWR_FLAG" H 7050 1350 50  0000 C CNN
+F 2 "" H 7050 1200 50  0001 C CNN
+F 3 "" H 7050 1200 50  0001 C CNN
+	1    7050 1200
 	1    0    0    -1
 $EndComp
@@
 L VCC #PWR020
 U 1 1 58EB3FDB
-P 7650 1350
-F 0 "#PWR020" H 7650 1200 50  0001 C CNN
-F 1 "VCC" H 7650 1500 50  0000 C CNN
-F 2 "" H 7650 1350 50  0001 C CNN
-F 3 "" H 7650 1350 50  0001 C CNN
-	1    7650 1350
+P 7700 1250
+F 0 "#PWR020" H 7700 1100 50  0001 C CNN
+F 1 "VCC" H 7700 1400 50  0000 C CNN
+F 2 "" H 7700 1250 50  0001 C CNN
+F 3 "" H 7700 1250 50  0001 C CNN
+	1    7700 1250
 	-1   0    0    1
 $EndComp
@@
 	1    0    0    -1
 $EndComp
-Text GLabel 7900 1300 2    30   Input ~ 0
+Text GLabel 8000 1200 2    30   Input ~ 0
 sense_pwr
 $Comp
 L PWR_FLAG #FLG038
 U 1 1 58F6EC3C
-P 7900 1300
-F 0 "#FLG038" H 7900 1375 50  0001 C CNN
-F 1 "PWR_FLAG" H 7900 1450 50  0000 C CNN
-F 2 "" H 7900 1300 50  0001 C CNN
-F 3 "" H 7900 1300 50  0001 C CNN
-	1    7900 1300
+P 8000 1200
+F 0 "#FLG038" H 8000 1275 50  0001 C CNN
+F 1 "PWR_FLAG" H 8000 1350 50  0000 C CNN
+F 2 "" H 8000 1200 50  0001 C CNN
+F 3 "" H 8000 1200 50  0001 C CNN
+	1    8000 1200
 	1    0    0    -1
 $EndComp
@@
 Text GLabel 8150 3200 0    30   Input ~ 0
 12V
-Text GLabel 7650 1200 1    30   Input ~ 0
+Text GLabel 7700 1100 1    30   Input ~ 0
 24V
-Text GLabel 7050 1350 0    30   Input ~ 0
+Text GLabel 7050 1250 0    30   Input ~ 0
 12V
 $Comp
 L PWR_FLAG #FLG040
 U 1 1 5934D9E0
-P 7450 1300
-F 0 "#FLG040" H 7450 1375 50  0001 C CNN
-F 1 "PWR_FLAG" H 7450 1450 50  0000 C CNN
-F 2 "" H 7450 1300 50  0001 C CNN
-F 3 "" H 7450 1300 50  0001 C CNN
-	1    7450 1300
+P 7500 1200
+F 0 "#FLG040" H 7500 1275 50  0001 C CNN
+F 1 "PWR_FLAG" H 7500 1350 50  0000 C CNN
+F 2 "" H 7500 1200 50  0001 C CNN
+F 3 "" H 7500 1200 50  0001 C CNN
+	1    7500 1200
 	1    0    0    -1
 $EndComp
@@
 	5700 12950 5700 13000
 Wire Wire Line
-	7050 1300 7050 1350
-Wire Wire Line
-	7650 1200 7650 1350
-Wire Wire Line
-	7450 1300 7650 1300
-Connection ~ 7650 1300
+	7050 1200 7050 1250
+Wire Wire Line
+	7700 1100 7700 1250
+Wire Wire Line
+	7500 1200 7700 1200
+Connection ~ 7700 1200
 Wire Notes Line
 	700  14000 6500 14000
@@
 L PWR_FLAG #FLG048
 U 1 1 59722FC4
-P 7550 1800
-F 0 "#FLG048" H 7550 1875 50  0001 C CNN
-F 1 "PWR_FLAG" H 7550 1950 50  0000 C CNN
-F 2 "" H 7550 1800 50  0001 C CNN
-F 3 "" H 7550 1800 50  0001 C CNN
-	1    7550 1800
-	1    0    0    -1
-$EndComp
-Text GLabel 7550 1800 3    30   Input ~ 0
+P 7600 1800
+F 0 "#FLG048" H 7600 1875 50  0001 C CNN
+F 1 "PWR_FLAG" H 7600 1950 50  0000 C CNN
+F 2 "" H 7600 1800 50  0001 C CNN
+F 3 "" H 7600 1800 50  0001 C CNN
+	1    7600 1800
+	1    0    0    -1
+$EndComp
+Text GLabel 7600 1800 0    30   Input ~ 0
 myRIO_12V
 $Comp
 L PWR_FLAG #FLG049
 U 1 1 59722053
-P 7950 1800
-F 0 "#FLG049" H 7950 1875 50  0001 C CNN
-F 1 "PWR_FLAG" H 7950 1950 50  0000 C CNN
-F 2 "" H 7950 1800 50  0001 C CNN
-F 3 "" H 7950 1800 50  0001 C CNN
-	1    7950 1800
-	1    0    0    -1
-$EndComp
-Text GLabel 7950 1800 3    39   Input ~ 0
+P 8150 1800
+F 0 "#FLG049" H 8150 1875 50  0001 C CNN
+F 1 "PWR_FLAG" H 8150 1950 50  0000 C CNN
+F 2 "" H 8150 1800 50  0001 C CNN
+F 3 "" H 8150 1800 50  0001 C CNN
+	1    8150 1800
+	1    0    0    -1
+$EndComp
+Text GLabel 8150 1800 0    39   Input ~ 0
 battery+fuse
 $Comp
@@
 	1    0    0    -1
 $EndComp
-Text GLabel 7150 1800 3    39   Input ~ 0
+Text GLabel 7150 1800 0    39   Input ~ 0
 battery
 $Comp
@@
 main_laser2
 NoConn ~ 22050 950
+$Comp
+L C C8
+U 1 1 59783929
+P 8150 1950
+F 0 "C8" H 8175 2050 50  0000 L CNN
+F 1 "C" H 8175 1850 50  0000 L CNN
+F 2 "Capacitors_THT:CP_Radial_D5.0mm_P2.50mm" H 8188 1800 50  0001 C CNN
+F 3 "" H 8150 1950 50  0001 C CNN
+	1    8150 1950
+	1    0    0    -1
+$EndComp
+$Comp
+L C C5
+U 1 1 5978666D
+P 7600 1950
+F 0 "C5" H 7625 2050 50  0000 L CNN
+F 1 "C" H 7625 1850 50  0000 L CNN
+F 2 "Capacitors_THT:CP_Radial_D5.0mm_P2.50mm" H 7638 1800 50  0001 C CNN
+F 3 "" H 7600 1950 50  0001 C CNN
+	1    7600 1950
+	1    0    0    -1
+$EndComp
+$Comp
+L C C3
+U 1 1 59786811
+P 7150 1950
+F 0 "C3" H 7175 2050 50  0000 L CNN
+F 1 "C" H 7175 1850 50  0000 L CNN
+F 2 "Capacitors_THT:CP_Radial_D5.0mm_P2.50mm" H 7188 1800 50  0001 C CNN
+F 3 "" H 7150 1950 50  0001 C CNN
+	1    7150 1950
+	1    0    0    -1
+$EndComp
+$Comp
+L C C6
+U 1 1 597869BE
+P 8000 1350
+F 0 "C6" H 8025 1450 50  0000 L CNN
+F 1 "C" H 8025 1250 50  0000 L CNN
+F 2 "Capacitors_THT:CP_Radial_D5.0mm_P2.50mm" H 8038 1200 50  0001 C CNN
+F 3 "" H 8000 1350 50  0001 C CNN
+	1    8000 1350
+	1    0    0    -1
+$EndComp
+$Comp
+L C C4
+U 1 1 59786B84
+P 7500 1350
+F 0 "C4" H 7525 1450 50  0000 L CNN
+F 1 "C" H 7525 1250 50  0000 L CNN
+F 2 "Capacitors_THT:CP_Radial_D5.0mm_P2.50mm" H 7538 1200 50  0001 C CNN
+F 3 "" H 7500 1350 50  0001 C CNN
+	1    7500 1350
+	1    0    0    -1
+$EndComp
+$Comp
+L C C2
+U 1 1 59786D3B
+P 7050 1400
+F 0 "C2" H 7075 1500 50  0000 L CNN
+F 1 "C" H 7075 1300 50  0000 L CNN
+F 2 "Capacitors_THT:CP_Radial_D5.0mm_P2.50mm" H 7088 1250 50  0001 C CNN
+F 3 "" H 7050 1400 50  0001 C CNN
+	1    7050 1400
+	1    0    0    -1
+$EndComp
+Wire Wire Line
+	7150 1500 8000 1500
+Wire Wire Line
+	7150 1550 7150 1500
+Wire Wire Line
+	6650 1550 7150 1550
+Connection ~ 7500 1500
+Connection ~ 6650 1550
+Connection ~ 7050 1550
+Wire Wire Line
+	6800 2100 8150 2100
+Connection ~ 7600 2100
+Wire Wire Line
+	6800 2100 6800 1750
+Wire Wire Line
+	6800 1750 6650 1750
+Connection ~ 7150 2100
+$Comp
+L C C7
+U 1 1 5978A2F0
+P 8000 3000
+F 0 "C7" H 8025 3100 50  0000 L CNN
+F 1 "C" H 8025 2900 50  0000 L CNN
+F 2 "Capacitors_THT:CP_Radial_D5.0mm_P2.50mm" H 8038 2850 50  0001 C CNN
+F 3 "" H 8000 3000 50  0001 C CNN
+	1    8000 3000
+	0    1    1    0
+$EndComp
+$Comp
+L C C1
+U 1 1 5978A917
+P 6550 2850
+F 0 "C1" H 6575 2950 50  0000 L CNN
+F 1 "C" H 6575 2750 50  0000 L CNN
+F 2 "Capacitors_THT:CP_Radial_D5.0mm_P2.50mm" H 6588 2700 50  0001 C CNN
+F 3 "" H 6550 2850 50  0001 C CNN
+	1    6550 2850
+	-1   0    0    1
+$EndComp
+$Comp
+L C C9
+U 1 1 5978C27D
+P 9600 2950
+F 0 "C9" H 9625 3050 50  0000 L CNN
+F 1 "C" H 9625 2850 50  0000 L CNN
+F 2 "Capacitors_THT:CP_Radial_D5.0mm_P2.50mm" H 9638 2800 50  0001 C CNN
+F 3 "" H 9600 2950 50  0001 C CNN
+	1    9600 2950
+	0    1    1    0
+$EndComp
+Text GLabel 6550 2700 2    30   Input ~ 0
+DGND
+Text GLabel 7850 3000 1    30   Input ~ 0
+DGND
+Text GLabel 9450 2950 1    30   Input ~ 0
+DGND
 $EndSCHEMATC

Commit message: traces for days
Parts:
- removed C8: C, Capacitors_THT:CP_Radial_D5.0mm_P2.50mm, symbol C
Changed lines of the file:
@@
 	22050 1450 22550 1450
 Wire Wire Line
-	22050 2150 22550 2150
+	22550 2150 22050 2150
 Wire Wire Line
 	3100 1650 3500 1650
@@
 	700  14000 700  12600
 Wire Wire Line
-	22550 2150 22550 1450
+	22550 1450 22550 2150
 Wire Wire Line
 	22550 1800 23050 1800
@@
 NoConn ~ 22050 950
 $Comp
-L C C8
-U 1 1 59783929
-P 8150 1950
-F 0 "C8" H 8175 2050 50  0000 L CNN
-F 1 "C" H 8175 1850 50  0000 L CNN
-F 2 "Capacitors_THT:CP_Radial_D5.0mm_P2.50mm" H 8188 1800 50  0001 C CNN
-F 3 "" H 8150 1950 50  0001 C CNN
-	1    8150 1950
-	1    0    0    -1
-$EndComp
-$Comp
 L C C5
 U 1 1 5978666D
@@
 Connection ~ 7050 1550
 Wire Wire Line
-	6800 2100 8150 2100
-Connection ~ 7600 2100
-Wire Wire Line
 	6800 2100 6800 1750
 Wire Wire Line
 	6800 1750 6650 1750
-Connection ~ 7150 2100
 $Comp
 L C C7
@@
 Text GLabel 9450 2950 1    30   Input ~ 0
 DGND
+Wire Wire Line
+	6800 2100 7650 2100
+Connection ~ 7150 2100
+Connection ~ 7600 2100
 $EndSCHEMATC

Commit message: made small changes according to feedback
Parts:
- added C?: C, Capacitors_THT:CP_Radial_D5.0mm_P2.50mm, symbol C
- added D?: D, Diodes_THT:D_DO-35_SOD27_P5.08mm_Vertical_AnodeUp, symbol D
- added R?: R, Resistors_THT:R_Axial_DIN0204_L3.6mm_D1.6mm_P5.08mm_Horizontal, symbol R
Connections:
- wire segments 215 -> 223
Other:
- moved on the sheet: D1, D2, Q1, Q2, R1, R2
Changed lines of the file:
@@
 L PN2222A Q1
 U 1 1 58DD3FFB
-P 13200 8750
-F 0 "Q1" H 13400 8825 50  0000 L CNN
-F 1 "PN2222A" H 13400 8750 50  0000 L CNN
-F 2 "TO_SOT_Packages_THT:TO-92_Inline_Narrow_Oval" H 13400 8675 50  0001 L CIN
-F 3 "" H 13200 8750 50  0000 L CNN
-	1    13200 8750
+P 13150 8900
+F 0 "Q1" H 13350 8975 50  0000 L CNN
+F 1 "PN2222A" H 13350 8900 50  0000 L CNN
+F 2 "TO_SOT_Packages_THT:TO-92_Inline_Narrow_Oval" H 13350 8825 50  0001 L CIN
+F 3 "" H 13150 8900 50  0000 L CNN
+	1    13150 8900
 	1    0    0    -1
 $EndComp
@@
 L R R1
 U 1 1 58DD4001
-P 13000 8900
-F 0 "R1" V 13080 8900 50  0000 C CNN
-F 1 "R" V 13000 8900 50  0000 C CNN
-F 2 "Resistors_THT:R_Axial_DIN0204_L3.6mm_D1.6mm_P5.08mm_Horizontal" V 12930 8900 50  0001 C CNN
-F 3 "" H 13000 8900 50  0000 C CNN
-	1    13000 8900
+P 12950 9050
+F 0 "R1" V 13030 9050 50  0000 C CNN
+F 1 "R" V 12950 9050 50  0000 C CNN
+F 2 "Resistors_THT:R_Axial_DIN0204_L3.6mm_D1.6mm_P5.08mm_Horizontal" V 12880 9050 50  0001 C CNN
+F 3 "" H 12950 9050 50  0000 C CNN
+	1    12950 9050
 	1    0    0    -1
 $EndComp
@@
 L GND #PWR07
 U 1 1 58DD4007
-P 13300 8950
-F 0 "#PWR07" H 13300 8700 50  0001 C CNN
-F 1 "GND" H 13300 8800 50  0000 C CNN
-F 2 "" H 13300 8950 50  0000 C CNN
-F 3 "" H 13300 8950 50  0000 C CNN
-	1    13300 8950
+P 13250 9100
+F 0 "#PWR07" H 13250 8850 50  0001 C CNN
+F 1 "GND" H 13250 8950 50  0000 C CNN
+F 2 "" H 13250 9100 50  0000 C CNN
+F 3 "" H 13250 9100 50  0000 C CNN
+	1    13250 9100
 	1    0    0    -1
 $EndComp
@@
 L D D1
 U 1 1 58DD400D
-P 13450 8400
-F 0 "D1" H 13450 8500 50  0000 C CNN
-F 1 "D" H 13450 8300 50  0000 C CNN
-F 2 "Diodes_THT:D_DO-35_SOD27_P5.08mm_Vertical_AnodeUp" H 13450 8400 50  0001 C CNN
-F 3 "" H 13450 8400 50  0000 C CNN
-	1    13450 8400
+P 13400 8550
+F 0 "D1" H 13400 8650 50  0000 C CNN
+F 1 "D" H 13400 8450 50  0000 C CNN
+F 2 "Diodes_THT:D_DO-35_SOD27_P5.08mm_Vertical_AnodeUp" H 13400 8550 50  0001 C CNN
+F 3 "" H 13400 8550 50  0000 C CNN
+	1    13400 8550
 	-1   0    0    1
 $EndComp
-Text GLabel 13600 8400 2    30   Input ~ 0
+Text GLabel 13550 8550 2    30   Input ~ 0
 5V
-Text GLabel 13000 9050 3    30   Input ~ 0
+Text GLabel 12950 9200 3    30   Input ~ 0
 2way_ctrl_1
-Text GLabel 12900 8550 3    30   Input ~ 0
+Text GLabel 12850 8700 3    30   Input ~ 0
 2way_ctrl_1_coil-
 $Comp
 L PN2222A Q2
 U 1 1 58DD4019
-P 14300 8750
-F 0 "Q2" H 14500 8825 50  0000 L CNN
-F 1 "PN2222A" H 14500 8750 50  0000 L CNN
-F 2 "TO_SOT_Packages_THT:TO-92_Inline_Narrow_Oval" H 14500 8675 50  0001 L CIN
-F 3 "" H 14300 8750 50  0000 L CNN
-	1    14300 8750
+P 14250 8900
+F 0 "Q2" H 14450 8975 50  0000 L CNN
+F 1 "PN2222A" H 14450 8900 50  0000 L CNN
+F 2 "TO_SOT_Packages_THT:TO-92_Inline_Narrow_Oval" H 14450 8825 50  0001 L CIN
+F 3 "" H 14250 8900 50  0000 L CNN
+	1    14250 8900
 	1    0    0    -1
 $EndComp
@@
 L R R2
 U 1 1 58DD401F
-P 14100 8900
-F 0 "R2" V 14180 8900 50  0000 C CNN
-F 1 "R" V 14100 8900 50  0000 C CNN
-F 2 "Resistors_THT:R_Axial_DIN0204_L3.6mm_D1.6mm_P5.08mm_Horizontal" V 14030 8900 50  0001 C CNN
-F 3 "" H 14100 8900 50  0000 C CNN
-	1    14100 8900
+P 14050 9050
+F 0 "R2" V 14130 9050 50  0000 C CNN
+F 1 "R" V 14050 9050 50  0000 C CNN
+F 2 "Resistors_THT:R_Axial_DIN0204_L3.6mm_D1.6mm_P5.08mm_Horizontal" V 13980 9050 50  0001 C CNN
+F 3 "" H 14050 9050 50  0000 C CNN
+	1    14050 9050
 	1    0    0    -1
 $EndComp
@@
 L GND #PWR08
 U 1 1 58DD4025
-P 14400 8950
-F 0 "#PWR08" H 14400 8700 50  0001 C CNN
-F 1 "GND" H 14400 8800 50  0000 C CNN
-F 2 "" H 14400 8950 50  0000 C CNN
-F 3 "" H 14400 8950 50  0000 C CNN
-	1    14400 8950
+P 14350 9100
+F 0 "#PWR08" H 14350 8850 50  0001 C CNN
+F 1 "GND" H 14350 8950 50  0000 C CNN
+F 2 "" H 14350 9100 50  0000 C CNN
+F 3 "" H 14350 9100 50  0000 C CNN
+	1    14350 9100
 	1    0    0    -1
 $EndComp
@@
 L D D2
 U 1 1 58DD402B
-P 14550 8400
-F 0 "D2" H 14550 8500 50  0000 C CNN
-F 1 "D" H 14550 8300 50  0000 C CNN
-F 2 "Diodes_THT:D_DO-35_SOD27_P5.08mm_Vertical_AnodeUp" H 14550 8400 50  0001 C CNN
-F 3 "" H 14550 8400 50  0000 C CNN
-	1    14550 8400
+P 14500 8550
+F 0 "D2" H 14500 8650 50  0000 C CNN
+F 1 "D" H 14500 8450 50  0000 C CNN
+F 2 "Diodes_THT:D_DO-35_SOD27_P5.08mm_Vertical_AnodeUp" H 14500 8550 50  0001 C CNN
+F 3 "" H 14500 8550 50  0000 C CNN
+	1    14500 8550
 	-1   0    0    1
 $EndComp
-Text GLabel 14700 8400 2    30   Input ~ 0
+Text GLabel 14650 8550 2    30   Input ~ 0
 5V
-Text GLabel 14100 9050 3    30   Input ~ 0
+Text GLabel 14050 9200 3    30   Input ~ 0
 2way_ctrl_2
-Text GLabel 14000 8550 3    30   Input ~ 0
+Text GLabel 13950 8700 3    30   Input ~ 0
 2way_ctrl_2_coil-
 Text Notes 14300 8100 2    99   ~ 0
@@
 	16400 -800 25550 -800
 Wire Wire Line
-	13300 8400 13300 8550
-Wire Wire Line
-	12900 8550 12900 8400
-Wire Wire Line
-	12900 8400 13300 8400
-Wire Wire Line
-	14400 8400 14400 8550
-Wire Wire Line
-	14000 8550 14000 8400
-Wire Wire Line
-	14000 8400 14400 8400
+	13250 8550 13250 8700
+Wire Wire Line
+	12850 8700 12850 8550
+Wire Wire Line
+	12850 8550 13250 8550
+Wire Wire Line
+	14350 8550 14350 8700
+Wire Wire Line
+	13950 8700 13950 8550
+Wire Wire Line
+	13950 8550 14350 8550
 Wire Wire Line
 	18250 6100 18250 6250
@@
 Connection ~ 7150 2100
 Connection ~ 7600 2100
+$Comp
+L R R?
+U 1 1 597F3813
+P 13950 7900
+F 0 "R?" V 14030 7900 50  0000 C CNN
+F 1 "R" V 13950 7900 50  0000 C CNN
+F 2 "Resistors_THT:R_Axial_DIN0204_L3.6mm_D1.6mm_P5.08mm_Horizontal" V 13880 7900 50  0001 C CNN
+F 3 "" H 13950 7900 50  0000 C CNN
+	1    13950 7900
+	0    1    1    0
+$EndComp
+Wire Wire Line
+	13700 7500 13700 7600
+Wire Wire Line
+	13700 7600 13250 7600
+Wire Wire Line
+	13250 7600 13250 7900
+Wire Wire Line
+	13250 7900 13800 7900
+$Comp
+L C C?
+U 1 1 597F6179
+P 14250 7900
+F 0 "C?" H 14275 8000 50  0000 L CNN
+F 1 "C" H 14275 7800 50  0000 L CNN
+F 2 "Capacitors_THT:CP_Radial_D5.0mm_P2.50mm" H 14288 7750 50  0001 C CNN
+F 3 "" H 14250 7900 50  0001 C CNN
+	1    14250 7900
+	0    1    1    0
+$EndComp
+Wire Wire Line
+	14650 7500 14650 7550
+Wire Wire Line
+	14650 7550 15050 7550
+Wire Wire Line
+	15050 7550 15050 7900
+Wire Wire Line
+	15050 7900 14400 7900
+$Comp
+L D D?
+U 1 1 597FC3BB
+P 15050 8050
+F 0 "D?" H 15050 8150 50  0000 C CNN
+F 1 "D" H 15050 7950 50  0000 C CNN
+F 2 "Diodes_THT:D_DO-35_SOD27_P5.08mm_Vertical_AnodeUp" H 15050 8050 50  0001 C CNN
+F 3 "" H 15050 8050 50  0000 C CNN
+	1    15050 8050
+	0    1    1    0
+$EndComp
+$Comp
+L GND #PWR?
+U 1 1 597FD891
+P 15050 8200
+F 0 "#PWR?" H 15050 7950 50  0001 C CNN
+F 1 "GND" H 15050 8050 50  0000 C CNN
+F 2 "" H 15050 8200 50  0000 C CNN
+F 3 "" H 15050 8200 50  0000 C CNN
+	1    15050 8200
+	1    0    0    -1
+$EndComp
 $EndSCHEMATC

Commit message: made changes according to 7-31 feedback doc
Parts:
- gave numbers to parts that had none: 3
Connections:
- net labels removed: motor_ctrl
- no-connect marks 113 -> 115
Changed lines of the file:
@@
 NoConn ~ 9850 5900
 NoConn ~ 9850 6000
-Text GLabel 1850 4600 0    60   Input ~ 0
-motor_ctrl
 $Comp
 L stacked-DB9 U8
@@
 NoConn ~ 4700 12800
 NoConn ~ 4700 12900
-Text GLabel 5700 12800 2    60   Input ~ 0
-motor_ctrl
 Text GLabel 5700 12900 2    30   Input ~ 0
 24V
@@
 Wire Wire Line
 	10100 6050 10100 6150
-Text GLabel 2600 1150 0    30   Input ~ 0
+Text GLabel 1850 4600 0    30   Input ~ 0
 laser_digital2
 Text GLabel 5600 9950 0    30   Input ~ 0
@@
 Connection ~ 7600 2100
 $Comp
-L R R?
+L R R34
 U 1 1 597F3813
 P 13950 7900
-F 0 "R?" V 14030 7900 50  0000 C CNN
+F 0 "R34" V 14030 7900 50  0000 C CNN
 F 1 "R" V 13950 7900 50  0000 C CNN
 F 2 "Resistors_THT:R_Axial_DIN0204_L3.6mm_D1.6mm_P5.08mm_Horizontal" V 13880 7900 50  0001 C CNN
@@
 	13250 7900 13800 7900
 $Comp
-L C C?
+L C C8
 U 1 1 597F6179
 P 14250 7900
-F 0 "C?" H 14275 8000 50  0000 L CNN
+F 0 "C8" H 14275 8000 50  0000 L CNN
 F 1 "C" H 14275 7800 50  0000 L CNN
 F 2 "Capacitors_THT:CP_Radial_D5.0mm_P2.50mm" H 14288 7750 50  0001 C CNN
@@
 	15050 7900 14400 7900
 $Comp
-L D D?
+L D D21
 U 1 1 597FC3BB
 P 15050 8050
-F 0 "D?" H 15050 8150 50  0000 C CNN
+F 0 "D21" H 15050 8150 50  0000 C CNN
 F 1 "D" H 15050 7950 50  0000 C CNN
 F 2 "Diodes_THT:D_DO-35_SOD27_P5.08mm_Vertical_AnodeUp" H 15050 8050 50  0001 C CNN
@@
 $EndComp
 $Comp
-L GND #PWR?
+L GND #PWR051
 U 1 1 597FD891
 P 15050 8200
-F 0 "#PWR?" H 15050 7950 50  0001 C CNN
+F 0 "#PWR051" H 15050 7950 50  0001 C CNN
 F 1 "GND" H 15050 8050 50  0000 C CNN
 F 2 "" H 15050 8200 50  0000 C CNN
@@
 	1    0    0    -1
 $EndComp
+NoConn ~ 2600 1150
+NoConn ~ 5700 12800
 $EndSCHEMATC

Commit message: commiting the schematic changes
Parts:
- removed S1: L101011MS02Q, footprints:L101011MS02Q, symbol L101011MS02Q
Connections:
- wire segments 223 -> 221
Other:
- note added: "check"
- note added: "check - why is the r connected to coil negative"
Changed lines of the file:
@@
 	-1   0    0    1
 $EndComp
-Text GLabel 22050 800  2    60   Input ~ 0
+Text GLabel 22050 950  2    60   Input ~ 0
 to_cap
 Text GLabel 21100 650  0    30   Input ~ 0
@@
 	1    0    0    -1
 $EndComp
-$Comp
-L L101011MS02Q S1
-U 1 1 59710165
-P 10050 1000
-F 0 "S1" H 10050 1050 60  0000 C CNN
-F 1 "L101011MS02Q" H 10100 1250 60  0000 C CNN
-F 2 "footprints:L101011MS02Q" H 10050 1000 60  0001 C CNN
-F 3 "" H 10050 1000 60  0001 C CNN
-	1    10050 1000
-	1    0    0    -1
-$EndComp
 Wire Wire Line
 	1400 3150 2550 3150
@@
 battery_sensor_input
 Wire Wire Line
-	9100 1100 9500 1100
+	9100 1100 10700 1100
 Text GLabel 10700 1100 2    39   Input ~ 0
 battery+fuse
@@
 Text GLabel 5600 10250 0    30   Input ~ 0
 main_laser2
-NoConn ~ 22050 950
+NoConn ~ 22050 800
 $Comp
 L C C5
@@
 	0    1    1    0
 $EndComp
-Wire Wire Line
-	13700 7500 13700 7600
-Wire Wire Line
-	13700 7600 13250 7600
-Wire Wire Line
-	13250 7600 13250 7900
-Wire Wire Line
-	13250 7900 13800 7900
 $Comp
 L C C8
@@
 NoConn ~ 2600 1150
 NoConn ~ 5700 12800
+Text Notes 8200 1350 0    60   ~ 0
+check
+Text Notes 13500 7250 0    60   ~ 0
+check - why is the r connected to coil negative
+Wire Wire Line
+	13700 7650 13700 7900
+Wire Wire Line
+	13700 7900 13800 7900
 $EndSCHEMATC

Commit message: donezo mcfunzo
Parts:
- removed D23: LED, LEDs:LED_D5.0mm, symbol LED-RESCUE-myrio_pcb
- added D23: LED, LEDs:LED_D5.0mm, symbol LED
- added T5: Phoenix_Contact_1935187, footprints:Phoenix_Contact_1935187, symbol Phoenix_Contact_1935187
Connections:
- net labels added: SolenoidGround, SolenoidPower
- wire segments 221 -> 222
Other:
- note removed: "check - why is the r connected to coil negative"
Changed lines of the file:
@@
 Text GLabel 13700 7500 0    30   Input ~ 0
 2way_ctrl_3_coil-
-Text GLabel 13700 7650 0    30   Input ~ 0
-24V_activation
-Text GLabel 13700 7350 0    30   Input ~ 0
-24V_activation
 $Comp
 L PN2222A Q3
@@
 Text GLabel 6700 11250 2    30   Input ~ 0
 2way_close_3
-Text GLabel 6700 11350 2    30   Input ~ 0
-DGND
 Text GLabel 6700 11450 2    30   Input ~ 0
 3way_port2_1
@@
 NoConn ~ -250 11600
 $Comp
-L LED-RESCUE-myrio_pcb D23
-U 1 1 596FFCA6
-P 9100 1300
-F 0 "D23" H 9100 1400 50  0000 C CNN
-F 1 "LED" H 9100 1200 50  0000 C CNN
-F 2 "LEDs:LED_D5.0mm" H 9100 1300 50  0001 C CNN
-F 3 "" H 9100 1300 50  0000 C CNN
-	1    9100 1300
-	0    -1   -1   0
-$EndComp
-$Comp
 L R R21
 U 1 1 597018D1
@@
 Text Notes 8200 1350 0    60   ~ 0
 check
-Text Notes 13500 7250 0    60   ~ 0
-check - why is the r connected to coil negative
 Wire Wire Line
 	13700 7650 13700 7900
 Wire Wire Line
 	13700 7900 13800 7900
+$Comp
+L LED D23
+U 1 1 598149AC
+P 9100 1350
+F 0 "D23" H 9100 1450 50  0000 C CNN
+F 1 "LED" H 9100 1250 50  0000 C CNN
+F 2 "LEDs:LED_D5.0mm" H 9100 1350 50  0001 C CNN
+F 3 "" H 9100 1350 50  0001 C CNN
+	1    9100 1350
+	0    -1   -1   0
+$EndComp
+Wire Wire Line
+	9100 1100 9100 1200
+$Comp
+L Phoenix_Contact_1935187 T5
+U 1 1 59817211
+P 3400 -1650
+F 0 "T5" H 3600 -1550 60  0000 C CNN
+F 1 "Phoenix_Contact_1935187" H 3950 -1400 60  0000 C CNN
+F 2 "footprints:Phoenix_Contact_1935187" H 3400 -1650 60  0001 C CNN
+F 3 "" H 3400 -1650 60  0001 C CNN
+	1    3400 -1650
+	1    0    0    -1
+$EndComp
+Text GLabel 4450 -1450 3    30   Input ~ 0
+SolenoidPower
+$Comp
+L GND #PWR053
+U 1 1 59820BF0
+P 3750 -1450
+F 0 "#PWR053" H 3750 -1700 50  0001 C CNN
+F 1 "GND" H 3750 -1600 50  0000 C CNN
+F 2 "" H 3750 -1450 50  0001 C CNN
+F 3 "" H 3750 -1450 50  0001 C CNN
+	1    3750 -1450
+	1    0    0    -1
+$EndComp
+Text GLabel 3400 -1450 3    30   Input ~ 0
+12V
+Text GLabel 13700 7350 0    30   Input ~ 0
+SolenoidPower
+Text GLabel 13700 7650 0    30   Input ~ 0
+SolenoidPower
+Text GLabel 4100 -1450 3    30   Input ~ 0
+SolenoidGround
+Text GLabel 9750 1550 3    30   Input ~ 0
+SolenoidGround
+$Comp
+L PWR_FLAG #FLG?
+U 1 1 598311D7
+P 9750 1550
+F 0 "#FLG?" H 9750 1625 50  0001 C CNN
+F 1 "PWR_FLAG" H 9750 1700 50  0000 C CNN
+F 2 "" H 9750 1550 50  0001 C CNN
+F 3 "" H 9750 1550 50  0001 C CNN
+	1    9750 1550
+	1    0    0    -1
+$EndComp
+Text GLabel 6700 11350 2    30   Input ~ 0
+SolenoidGround
 $EndSCHEMATC
