File: myrio/myrio_pcb.sch (KiCad schematic (older format))
At the start: 139 parts, among them J1 CONN_02X03, J2 CONN_02X03, J3 CONN_02X03, J4 CONN_02X03, P1 CONN_02X17, P2 CONN_02X17, Q1 PN2222A, Q10 PN2222A, Q11 PN2222A, Q12 PN2222A, Q13 PN2222A, Q14 PN2222A, Q15 PN2222A, Q16 PN2222A, Q17 PN2222A, Q18 PN2222A, Q19 PN2222A, Q2 PN2222A, Q20 PN2222A, Q3 PN2222A, Q4 PN2222A, Q5 PN2222A, Q6 PN2222A, Q7 PN2222A, Q8 PN2222A, Q9 PN2222A, T1 Phoenix_Contact_1935187, T2 Phoenix_Contact_1935187, T3 Phoenix_Contact_1935187, T4 Phoenix_Contact_1935187, T5 Phoenix_Contact_1935187, U1 stacked-DB9, U10 INA219, U11 INA219, U13 INA219, U14 stacked-rj45-LED, U15 stacked-rj45-LED, U2 stacked-DB9, U3 stacked-rj45-LED, U4 stacked-rj45-LED, U5 stacked-rj45-LED, U6 BNO055, U7 stacked-rj45-LED, U8 stacked-DB9

Commit message: updated the schematic
Parts:
- removed C8: C, Capacitors_THT:CP_Radial_D5.0mm_P2.50mm, symbol C
- removed D21: D, Diodes_THT:D_DO-35_SOD27_P5.08mm_Vertical_AnodeUp, symbol D
- removed R34: R, Resistors_THT:R_Axial_DIN0204_L3.6mm_D1.6mm_P5.08mm_Horizontal, symbol R
Connections:
- net 24V_activation: now also RE8.5 (load1), RE8.6 (load2)
- net GND: now also U14.11
- net SolenoidGround: no longer names the net of T5.3 (pin3)
- net SolenoidGround: no longer U14.11
- removed net SolenoidPower: RE8.5 (load1), RE8.6 (load2), T5.4 (pin4)
- no-connect marks 115 -> 117
Other:
- note added: "Don't know what the 12V and Gnd signal is for here?"
Changed lines of the file:
@@
 Connection ~ 7150 2100
 Connection ~ 7600 2100
-$Comp
-L R R34
-U 1 1 597F3813
-P 13950 7900
-F 0 "R34" V 14030 7900 50  0000 C CNN
-F 1 "R" V 13950 7900 50  0000 C CNN
-F 2 "Resistors_THT:R_Axial_DIN0204_L3.6mm_D1.6mm_P5.08mm_Horizontal" V 13880 7900 50  0001 C CNN
-F 3 "" H 13950 7900 50  0000 C CNN
-	1    13950 7900
-	0    1    1    0
-$EndComp
-$Comp
-L C C8
-U 1 1 597F6179
-P 14250 7900
-F 0 "C8" H 14275 8000 50  0000 L CNN
-F 1 "C" H 14275 7800 50  0000 L CNN
-F 2 "Capacitors_THT:CP_Radial_D5.0mm_P2.50mm" H 14288 7750 50  0001 C CNN
-F 3 "" H 14250 7900 50  0001 C CNN
-	1    14250 7900
-	0    1    1    0
-$EndComp
-Wire Wire Line
-	14650 7500 14650 7550
-Wire Wire Line
-	14650 7550 15050 7550
-Wire Wire Line
-	15050 7550 15050 7900
-Wire Wire Line
-	15050 7900 14400 7900
-$Comp
-L D D21
-U 1 1 597FC3BB
-P 15050 8050
-F 0 "D21" H 15050 8150 50  0000 C CNN
-F 1 "D" H 15050 7950 50  0000 C CNN
-F 2 "Diodes_THT:D_DO-35_SOD27_P5.08mm_Vertical_AnodeUp" H 15050 8050 50  0001 C CNN
-F 3 "" H 15050 8050 50  0000 C CNN
-	1    15050 8050
-	0    1    1    0
-$EndComp
-$Comp
-L GND #PWR051
-U 1 1 597FD891
-P 15050 8200
-F 0 "#PWR051" H 15050 7950 50  0001 C CNN
-F 1 "GND" H 15050 8050 50  0000 C CNN
-F 2 "" H 15050 8200 50  0000 C CNN
-F 3 "" H 15050 8200 50  0000 C CNN
-	1    15050 8200
-	1    0    0    -1
-$EndComp
 NoConn ~ 2600 1150
 NoConn ~ 5700 12800
 Text Notes 8200 1350 0    60   ~ 0
 check
-Wire Wire Line
-	13700 7650 13700 7900
-Wire Wire Line
-	13700 7900 13800 7900
 $Comp
 L LED D23
@@
 	1    0    0    -1
 $EndComp
-Text GLabel 4450 -1450 3    30   Input ~ 0
-SolenoidPower
 $Comp
 L GND #PWR053
@@
 12V
 Text GLabel 13700 7350 0    30   Input ~ 0
-SolenoidPower
+24V_activation
 Text GLabel 13700 7650 0    30   Input ~ 0
-SolenoidPower
-Text GLabel 4100 -1450 3    30   Input ~ 0
-SolenoidGround
-Text GLabel 9750 1550 3    30   Input ~ 0
-SolenoidGround
-$Comp
-L PWR_FLAG #FLG?
-U 1 1 598311D7
-P 9750 1550
-F 0 "#FLG?" H 9750 1625 50  0001 C CNN
-F 1 "PWR_FLAG" H 9750 1700 50  0000 C CNN
-F 2 "" H 9750 1550 50  0001 C CNN
-F 3 "" H 9750 1550 50  0001 C CNN
-	1    9750 1550
-	1    0    0    -1
-$EndComp
+24V_activation
 Text GLabel 6700 11350 2    30   Input ~ 0
-SolenoidGround
+DGND
+NoConn ~ 4100 -1450
+NoConn ~ 4450 -1450
+Text Notes 2400 -2100 0    60   ~ 0
+Don't know what the 12V and Gnd signal is for here?
 $EndSCHEMATC

Commit message: done for real this time
Parts:
- removed T5: Phoenix_Contact_1935187, footprints:Phoenix_Contact_1935187, symbol Phoenix_Contact_1935187
Connections:
- no-connect marks 117 -> 115
Other:
- note removed: "Don't know what the 12V and Gnd signal is for here?"
Changed lines of the file:
@@
 Wire Wire Line
 	9100 1100 9100 1200
-$Comp
-L Phoenix_Contact_1935187 T5
-U 1 1 59817211
-P 3400 -1650
-F 0 "T5" H 3600 -1550 60  0000 C CNN
-F 1 "Phoenix_Contact_1935187" H 3950 -1400 60  0000 C CNN
-F 2 "footprints:Phoenix_Contact_1935187" H 3400 -1650 60  0001 C CNN
-F 3 "" H 3400 -1650 60  0001 C CNN
-	1    3400 -1650
-	1    0    0    -1
-$EndComp
-$Comp
-L GND #PWR053
-U 1 1 59820BF0
-P 3750 -1450
-F 0 "#PWR053" H 3750 -1700 50  0001 C CNN
-F 1 "GND" H 3750 -1600 50  0000 C CNN
-F 2 "" H 3750 -1450 50  0001 C CNN
-F 3 "" H 3750 -1450 50  0001 C CNN
-	1    3750 -1450
-	1    0    0    -1
-$EndComp
-Text GLabel 3400 -1450 3    30   Input ~ 0
-12V
 Text GLabel 13700 7350 0    30   Input ~ 0
 24V_activation
@@
 Text GLabel 6700 11350 2    30   Input ~ 0
 DGND
-NoConn ~ 4100 -1450
-NoConn ~ 4450 -1450
-Text Notes 2400 -2100 0    60   ~ 0
-Don't know what the 12V and Gnd signal is for here?
 $EndSCHEMATC
