File: sensorPcbs/pod_health_thermopile/pod_health_thermopile.kicad_pcb (KiCad board)
At the start: 2 copper layers, 45.7 x 35.6 mm, 8 parts, among them J1 RJ45, U1 TMP007

Commit message: added all the ferkin new ethernet shields to the sensor pcbs
Parts:
- removed J1: RJ45, Connectors:RJ45_8
- added E1: RJE71-188-1401-ND, footprints:RJE71-188-1401-ND, F.Cu at (164.5, 81.0)
Connections:
- U1 pad 1: Net-(J1-Pad1) -> vcc
- U1 pad 2: Net-(J1-Pad2) -> gnd
- U1 pad 3: Net-(J1-Pad6) -> sda
- U1 pad 4: Net-(J1-Pad3) -> scl
Routing:
- net sda: track 0.00 -> 23.7 mm
- net scl: track 0.00 -> 22.0 mm
- net vcc: track 0.00 -> 21.3 mm
- net Net-(J1-Pad3): track 16.1 -> 0.00 mm
- net gnd: track 0.00 -> 14.9 mm
- net Net-(J1-Pad1): track 11.7 -> 0.00 mm
- net Net-(J1-Pad6): track 9.72 -> 0.00 mm
- net Net-(J1-Pad2): track 8.67 -> 0.00 mm
