File: sensorPcbs/pod_health_laser/pod_health_laser.kicad_pcb (KiCad board)
At the start: 2 copper layers, 77.5 x 35.6 mm, 10 parts, among them J1 RJ45, U1 laser_sensor

Commit message: added all the ferkin new ethernet shields to the sensor pcbs
Parts:
- removed J1: RJ45, Connectors:RJ45_8
- added E1: RJE71-188-1401-ND, footprints:RJE71-188-1401-ND, F.Cu at (172.6, 94.6)
Routing:
- net Net-(E1-Pad3): track 10.5 -> 31.1 mm
- net Net-(E1-Pad1): track 9.42 -> 23.7 mm
- net Net-(E1-Pad2): track 7.40 -> 11.1 mm
Changed lines of the file:
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@@
     (links 3)
     (no_connects 0)
-    (area 153.384999 84.877 231.215001 120.915)
+    (area 153.594999 85.014999 231.215001 120.725001)
     (thickness 1.6)
     (drawings 6)
-    (tracks 6)
+    (tracks 20)
     (zones 0)
     (modules 10)
@@
   )
   (net 0 "")
-  (net 1 "Net-(J1-Pad1)")
-  (net 2 "Net-(J1-Pad2)")
-  (net 3 "Net-(J1-Pad3)")
-  (net 4 "Net-(J1-Pad4)")
-  (net 5 "Net-(J1-Pad5)")
-  (net 6 "Net-(J1-Pad6)")
-  (net 7 "Net-(J1-Pad7)")
-  (net 8 "Net-(J1-Pad8)")
+  (net 1 "Net-(E1-Pad1)")
+  (net 2 "Net-(E1-Pad2)")
+  (net 3 "Net-(E1-Pad3)")
+  (net 4 "Net-(E1-Pad4)")
+  (net 5 "Net-(E1-Pad5)")
+  (net 6 "Net-(E1-Pad6)")
+  (net 7 "Net-(E1-Pad8)")
+  (net 8 "Net-(E1-Pad7)")
   (net_class Default "This is the default net class."
     (clearance 0.2)
@@
     (uvia_dia 0.3)
     (uvia_drill 0.1)
-    (add_net "Net-(J1-Pad1)")
-    (add_net "Net-(J1-Pad2)")
-    (add_net "Net-(J1-Pad3)")
-    (add_net "Net-(J1-Pad4)")
-    (add_net "Net-(J1-Pad5)")
-    (add_net "Net-(J1-Pad6)")
-    (add_net "Net-(J1-Pad7)")
-    (add_net "Net-(J1-Pad8)")
-  )
-  (module Connectors:RJ45_8 (layer F.Cu)
-    (at 170.18 99.06 270)
-    (tags RJ45)
-    (fp_text reference J1 (at 4.7 11.18 270) (layer F.SilkS)
-      (effects (font (size 1 1) (thickness 0.15)))
-    )
-    (fp_text value RJ45 (at 4.59 6.25 270) (layer F.Fab)
-      (effects (font (size 1 1) (thickness 0.15)))
-    )
-    (fp_line (start -3.17 14.22) (end 12.07 14.22) (layer F.SilkS) (width 0.12))
-    (fp_line (start 12.07 -3.81) (end 12.06 5.18) (layer F.SilkS) (width 0.12))
-    (fp_line (start 12.07 -3.81) (end -3.17 -3.81) (layer F.SilkS) (width 0.12))
-    (fp_line (start -3.17 -3.81) (end -3.17 5.19) (layer F.SilkS) (width 0.12))
-    (fp_line (start 12.06 7.52) (end 12.07 14.22) (layer F.SilkS) (width 0.12))
-    (fp_line (start -3.17 7.51) (end -3.17 14.22) (layer F.SilkS) (width 0.12))
-    (fp_line (start -3.56 -4.06) (end 12.46 -4.06) (layer F.CrtYd) (width 0.05))
-    (fp_line (start -3.56 -4.06) (end -3.56 14.47) (layer F.CrtYd) (width 0.05))
-    (fp_line (start 12.46 14.47) (end 12.46 -4.06) (layer F.CrtYd) (width 0.05))
-    (fp_line (start 12.46 14.47) (end -3.56 14.47) (layer F.CrtYd) (width 0.05))
-    (pad Hole np_thru_hole circle (at 10.38 6.35 270) (size 3.65 3.65) (drill 3.25) (layers *.Cu *.SilkS *.Mask))
-    (pad Hole np_thru_hole circle (at -1.49 6.35 270) (size 3.65 3.65) (drill 3.25) (layers *.Cu *.SilkS *.Mask))
-    (pad 1 thru_hole rect (at 0 0 270) (size 1.5 1.5) (drill 0.9) (layers *.Cu *.Mask)
-      (net 1 "Net-(J1-Pad1)"))
-    (pad 2 thru_hole circle (at 1.27 -2.54 270) (size 1.5 1.5) (drill 0.9) (layers *.Cu *.Mask)
-      (net 2 "Net-(J1-Pad2)"))
-    (pad 3 thru_hole circle (at 2.54 0 270) (size 1.5 1.5) (drill 0.9) (layers *.Cu *.Mask)
-      (net 3 "Net-(J1-Pad3)"))
-    (pad 4 thru_hole circle (at 3.81 -2.54 270) (size 1.5 1.5) (drill 0.9) (layers *.Cu *.Mask)
-      (net 4 "Net-(J1-Pad4)"))
-    (pad 5 thru_hole circle (at 5.08 0 270) (size 1.5 1.5) (drill 0.9) (layers *.Cu *.Mask)
-      (net 5 "Net-(J1-Pad5)"))
-    (pad 6 thru_hole circle (at 6.35 -2.54 270) (size 1.5 1.5) (drill 0.9) (layers *.Cu *.Mask)
-      (net 6 "Net-(J1-Pad6)"))
-    (pad 7 thru_hole circle (at 7.62 0 270) (size 1.5 1.5) (drill 0.9) (layers *.Cu *.Mask)
-      (net 7 "Net-(J1-Pad7)"))
-    (pad 8 thru_hole circle (at 8.89 -2.54 270) (size 1.5 1.5) (drill 0.9) (layers *.Cu *.Mask)
-      (net 8 "Net-(J1-Pad8)"))
-    (model Connectors.3dshapes/RJ45_8.wrl
-      (at (xyz 0.18 -0.25 0))
-      (scale (xyz 0.4 0.4 0.4))
-      (rotate (xyz 0 0 0))
-    )
+    (add_net "Net-(E1-Pad1)")
+    (add_net "Net-(E1-Pad2)")
+    (add_net "Net-(E1-Pad3)")
+    (add_net "Net-(E1-Pad4)")
+    (add_net "Net-(E1-Pad5)")
+    (add_net "Net-(E1-Pad6)")
+    (add_net "Net-(E1-Pad7)")
+    (add_net "Net-(E1-Pad8)")
   )
   (module laser_sensor:laser_sensor (layer F.Cu)
@@
     )
     (pad 1 thru_hole circle (at 2.54 2.54) (size 1.524 1.524) (drill 0.762) (layers *.Cu *.Mask)
-      (net 3 "Net-(J1-Pad3)"))
+      (net 3 "Net-(E1-Pad3)"))
     (pad 2 thru_hole circle (at 2.54 0) (size 1.524 1.524) (drill 0.762) (layers *.Cu *.Mask)
-      (net 2 "Net-(J1-Pad2)"))
+      (net 2 "Net-(E1-Pad2)"))
     (pad 3 thru_hole circle (at 2.54 -2.54) (size 1.524 1.524) (drill 0.762) (layers *.Cu *.Mask)
-      (net 1 "Net-(J1-Pad1)"))
+      (net 1 "Net-(E1-Pad1)"))
   )
   (module Connectors:1pin (layer F.Cu)
@@
     (fp_circle (center 0 0) (end 0 -2.286) (layer F.SilkS) (width 0.12))
     (pad 1 thru_hole circle (at 0 0) (size 4.064 4.064) (drill 3.048) (layers *.Cu *.Mask))
+  )
+  (module footprints:RJE71-188-1401-ND (layer F.Cu)
+    (at 172.6 94.6 270)
+    (fp_text reference E1 (at 8.47 11.9 270) (layer F.SilkS)
+      (effects (font (size 1 1) (thickness 0.15)))
+    )
+    (fp_text value RJE71-188-1401-ND (at 14.8 9.7 360) (layer F.Fab)
+      (effects (font (size 1 1) (thickness 0.15)))
+    )
+    (fp_text user SOCKET (at 7.6 16 270) (layer F.SilkS)
+      (effects (font (size 1 1) (thickness 0.15)))
+    )
+    (fp_line (start 16.2 0) (end 16.2 20.7) (layer F.SilkS) (width 0.25))
+    (fp_line (start 0 20.7) (end 16.2 20.7) (layer F.SilkS) (width 0.25))
+    (fp_line (start 0 0) (end 16.2 0) (layer F.SilkS) (width 0.25))
+    (fp_line (start 0 0) (end 0 20.7) (layer F.SilkS) (width 0.25))
+    (pad 1 thru_hole circle (at 11.67 5.45 270) (size 1.6 1.6) (drill 0.95) (layers *.Cu *.Mask)
+      (net 1 "Net-(E1-Pad1)"))
+    (pad 2 thru_hole circle (at 10.65 3.67 270) (size 1.6 1.6) (drill 0.95) (layers *.Cu *.Mask)
+      (net 2 "Net-(E1-Pad2)"))
+    (pad 3 thru_hole circle (at 9.63 5.45 270) (size 1.6 1.6) (drill 0.95) (layers *.Cu *.Mask)
+      (net 3 "Net-(E1-Pad3)"))
+    (pad 4 thru_hole circle (at 8.61 3.67 270) (size 1.6 1.6) (drill 0.95) (layers *.Cu *.Mask)
+      (net 4 "Net-(E1-Pad4)"))
+    (pad 5 thru_hole circle (at 7.59 5.45 270) (size 1.6 1.6) (drill 0.95) (layers *.Cu *.Mask)
+      (net 5 "Net-(E1-Pad5)"))
+    (pad 6 thru_hole circle (at 6.57 3.67 270) (size 1.6 1.6) (drill 0.95) (layers *.Cu *.Mask)
+      (net 6 "Net-(E1-Pad6)"))
+    (pad "" thru_hole oval (at -1.82 11.72 270) (size 1.8 3.2) (drill oval 1.1 2.5) (layers *.Cu *.Mask))
+    (pad "" thru_hole oval (at 18.02 11.72 270) (size 1.8 3.2) (drill oval 1.1 2.5) (layers *.Cu *.Mask))
+    (pad 8 thru_hole circle (at 4.53 3.67 270) (size 1.6 1.6) (drill 0.95) (layers *.Cu *.Mask)
+      (net 7 "Net-(E1-Pad8)"))
+    (pad 7 thru_hole circle (at 5.55 5.45 270) (size 1.6 1.6) (drill 0.95) (layers *.Cu *.Mask)
+      (net 8 "Net-(E1-Pad7)"))
   )
   (gr_line (start 231.14 85.09) (end 229.87 85.09) (angle 90) (layer Edge.Cuts) (width 0.15))
@@
   (gr_line (start 153.67 85.09) (end 153.67 119.38) (angle 90) (layer Edge.Cuts) (width 0.15))
   (gr_line (start 229.87 85.09) (end 153.67 85.09) (angle 90) (layer Edge.Cuts) (width 0.15))
-  (segment (start 170.18 99.06) (end 177.8 99.06) (width 0.25) (layer F.Cu) (net 1))
-  (segment (start 177.8 99.06) (end 179.07 100.33) (width 0.25) (layer F.Cu) (net 1))
-  (segment (start 172.72 100.33) (end 176.53 100.33) (width 0.25) (layer F.Cu) (net 2))
-  (segment (start 176.53 100.33) (end 179.07 102.87) (width 0.25) (layer F.Cu) (net 2))
-  (segment (start 170.18 101.6) (end 175.26 101.6) (width 0.25) (layer F.Cu) (net 3))
-  (segment (start 175.26 101.6) (end 179.07 105.41) (width 0.25) (layer F.Cu) (net 3))
+  (segment (start 179.07 100.33) (end 181.13 100.33) (width 0.25) (layer F.Cu) (net 1) (status 400000))
+  (segment (start 168.18 107.3) (end 167.15 106.27) (width 0.25) (layer F.Cu) (net 1) (status 800000))
+  (segment (start 180.4 107.3) (end 168.18 107.3) (width 0.25) (layer F.Cu) (net 1))
+  (segment (start 182 105.7) (end 180.4 107.3) (width 0.25) (layer F.Cu) (net 1))
+  (segment (start 182 101.2) (end 182 105.7) (width 0.25) (layer F.Cu) (net 1))
+  (segment (start 181.13 100.33) (end 182 101.2) (width 0.25) (layer F.Cu) (net 1))
+  (segment (start 168.93 105.25) (end 172.75 105.25) (width 0.25) (layer F.Cu) (net 2) (status 400000))
+  (segment (start 175.13 102.87) (end 179.07 102.87) (width 0.25) (layer F.Cu) (net 2) (status 800000))
+  (segment (start 172.75 105.25) (end 175.13 102.87) (width 0.25) (layer F.Cu) (net 2))
+  (segment (start 167.15 104.23) (end 165.43 104.23) (width 0.25) (layer B.Cu) (net 3) (status 400000))
+  (segment (start 176.29 105.41) (end 179.07 105.41) (width 0.25) (layer B.Cu) (net 3) (status 800000))
+  (segment (start 175.7 106) (end 176.29 105.41) (width 0.25) (layer B.Cu) (net 3))
+  (segment (start 172 106) (end 175.7 106) (width 0.25) (layer B.Cu) (net 3))
+  (segment (start 171.2 105.2) (end 172 106) (width 0.25) (layer B.Cu) (net 3))
+  (segment (start 171.2 98.1) (end 171.2 105.2) (width 0.25) (layer B.Cu) (net 3))
+  (segment (start 170.5 97.4) (end 171.2 98.1) (width 0.25) (layer B.Cu) (net 3))
+  (segment (start 165.4 97.4) (end 170.5 97.4) (width 0.25) (layer B.Cu) (net 3))
+  (segment (start 164.3 98.5) (end 165.4 97.4) (width 0.25) (layer B.Cu) (net 3))
+  (segment (start 164.3 103.1) (end 164.3 98.5) (width 0.25) (layer B.Cu) (net 3))
+  (segment (start 165.43 104.23) (end 164.3 103.1) (width 0.25) (layer B.Cu) (net 3))
 )

Commit message: fixed the laser circuit
Parts:
- U1: footprint laser_sensor:laser_sensor -> laser_sensor:laser_sensor_new
- moved REF** 5.72 mm to (221.6, 95.2)
- moved REF** 5.72 mm to (221.6, 110.5)
Changed lines of the file:
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@@
-(kicad_pcb (version 4) (host pcbnew 4.0.6)
+(kicad_pcb (version 4) (host pcbnew 4.0.3-stable)
   (general
     (links 3)
@@
     (mod_text_size 1 1)
     (mod_text_width 0.15)
-    (pad_size 1.524 1.524)
-    (pad_drill 0.762)
+    (pad_size 3 3)
+    (pad_drill 2)
     (pad_to_mask_clearance 0.2)
     (aux_axis_origin 0 0)
@@
     (add_net "Net-(E1-Pad8)")
   )
-  (module laser_sensor:laser_sensor (layer F.Cu)
-    (at 176.53 102.87)
-    (fp_text reference U1 (at 15.24 2.54) (layer F.SilkS)
-      (effects (font (size 1 1) (thickness 0.15)))
-    )
-    (fp_text value laser_sensor (at 15.24 -2.54) (layer F.Fab)
-      (effects (font (size 1 1) (thickness 0.15)))
-    )
-    (fp_line (start 0 10.16) (end 0 -10.16) (layer F.SilkS) (width 0.15))
-    (fp_line (start 53.34 -10.16) (end 53.34 10.16) (layer F.SilkS) (width 0.15))
-    (fp_line (start 53.34 10.16) (end 49.53 10.16) (layer F.SilkS) (width 0.15))
-    (fp_line (start 0 -10.16) (end 53.34 -10.16) (layer F.SilkS) (width 0.15))
-    (fp_line (start 49.53 10.16) (end 0 10.16) (layer F.SilkS) (width 0.15))
-    (fp_text user VCC (at 7.62 -2.54) (layer F.SilkS)
-      (effects (font (size 1 1) (thickness 0.15)))
-    )
-    (fp_text user GND (at 7.62 0) (layer F.SilkS)
-      (effects (font (size 1 1) (thickness 0.15)))
-    )
-    (fp_text user DOUT (at 7.62 2.54) (layer F.SilkS)
-      (effects (font (size 1 1) (thickness 0.15)))
-    )
-    (pad 1 thru_hole circle (at 2.54 2.54) (size 1.524 1.524) (drill 0.762) (layers *.Cu *.Mask)
-      (net 3 "Net-(E1-Pad3)"))
-    (pad 2 thru_hole circle (at 2.54 0) (size 1.524 1.524) (drill 0.762) (layers *.Cu *.Mask)
-      (net 2 "Net-(E1-Pad2)"))
-    (pad 3 thru_hole circle (at 2.54 -2.54) (size 1.524 1.524) (drill 0.762) (layers *.Cu *.Mask)
-      (net 1 "Net-(E1-Pad1)"))
-  )
   (module Connectors:1pin (layer F.Cu)
     (at 156.21 88.9)
@@
     (fp_circle (center 0 0) (end 2.6 0) (layer F.CrtYd) (width 0.05))
     (fp_circle (center 0 0) (end 0 -2.286) (layer F.SilkS) (width 0.12))
-    (pad 1 thru_hole circle (at 0 0) (size 4.064 4.064) (drill 3.048) (layers *.Cu *.Mask))
+    (pad 1 thru_hole circle (at 0 0) (size 3 3) (drill 2) (layers *.Cu *.Mask))
   )
   (module Connectors:1pin (layer F.Cu)
@@
     (fp_circle (center 0 0) (end 2.6 0) (layer F.CrtYd) (width 0.05))
     (fp_circle (center 0 0) (end 0 -2.286) (layer F.SilkS) (width 0.12))
-    (pad 1 thru_hole circle (at 0 0) (size 4.064 4.064) (drill 3.048) (layers *.Cu *.Mask))
-  )
-  (module Connectors:1pin (layer F.Cu)
-    (at 227.33 95.25)
-    (descr "module 1 pin (ou trou mecanique de percage)")
-    (tags DEV)
-    (fp_text reference REF** (at 0 -3.048) (layer F.SilkS)
-      (effects (font (size 1 1) (thickness 0.15)))
-    )
-    (fp_text value 1pin (at 0 3) (layer F.Fab)
-      (effects (font (size 1 1) (thickness 0.15)))
-    )
-    (fp_circle (center 0 0) (end 2 0.8) (layer F.Fab) (width 0.1))
-    (fp_circle (center 0 0) (end 2.6 0) (layer F.CrtYd) (width 0.05))
-    (fp_circle (center 0 0) (end 0 -2.286) (layer F.SilkS) (width 0.12))
-    (pad 1 thru_hole circle (at 0 0) (size 4.064 4.064) (drill 3.048) (layers *.Cu *.Mask))
-  )
-  (module Connectors:1pin (layer F.Cu)
-    (at 227.33 110.49)
-    (descr "module 1 pin (ou trou mecanique de percage)")
-    (tags DEV)
-    (fp_text reference REF** (at 0 -3.048) (layer F.SilkS)
-      (effects (font (size 1 1) (thickness 0.15)))
-    )
-    (fp_text value 1pin (at 0 3) (layer F.Fab)
-      (effects (font (size 1 1) (thickness 0.15)))
-    )
-    (fp_circle (center 0 0) (end 2 0.8) (layer F.Fab) (width 0.1))
-    (fp_circle (center 0 0) (end 2.6 0) (layer F.CrtYd) (width 0.05))
-    (fp_circle (center 0 0) (end 0 -2.286) (layer F.SilkS) (width 0.12))
-    (pad 1 thru_hole circle (at 0 0) (size 4.064 4.064) (drill 3.048) (layers *.Cu *.Mask))
+    (pad 1 thru_hole circle (at 0 0) (size 3 3) (drill 2) (layers *.Cu *.Mask))
+  )
+  (module Connectors:1pin (layer F.Cu)
+    (at 221.615 95.25)
+    (descr "module 1 pin (ou trou mecanique de percage)")
+    (tags DEV)
+    (fp_text reference REF** (at 0 -3.048) (layer F.SilkS)
+      (effects (font (size 1 1) (thickness 0.15)))
+    )
+    (fp_text value 1pin (at 0 3) (layer F.Fab)
+      (effects (font (size 1 1) (thickness 0.15)))
+    )
+    (fp_circle (center 0 0) (end 2 0.8) (layer F.Fab) (width 0.1))
+    (fp_circle (center 0 0) (end 2.6 0) (layer F.CrtYd) (width 0.05))
+    (fp_circle (center 0 0) (end 0 -2.286) (layer F.SilkS) (width 0.12))
+    (pad 1 thru_hole circle (at 0 0) (size 3 3) (drill 2) (layers *.Cu *.Mask))
+  )
+  (module Connectors:1pin (layer F.Cu)
+    (at 221.615 110.49)
+    (descr "module 1 pin (ou trou mecanique de percage)")
+    (tags DEV)
+    (fp_text reference REF** (at 0 -3.048) (layer F.SilkS)
+      (effects (font (size 1 1) (thickness 0.15)))
+    )
+    (fp_text value 1pin (at 0 3) (layer F.Fab)
+      (effects (font (size 1 1) (thickness 0.15)))
+    )
+    (fp_circle (center 0 0) (end 2 0.8) (layer F.Fab) (width 0.1))
+    (fp_circle (center 0 0) (end 2.6 0) (layer F.CrtYd) (width 0.05))
+    (fp_circle (center 0 0) (end 0 -2.286) (layer F.SilkS) (width 0.12))
+    (pad 1 thru_hole circle (at 0 0) (size 3 3) (drill 2) (layers *.Cu *.Mask))
   )
   (module footprints:RJE71-188-1401-ND (layer F.Cu)
@@
       (net 8 "Net-(E1-Pad7)"))
   )
+  (module laser_sensor:laser_sensor_new (layer F.Cu)
+    (at 176.53 102.87)
+    (fp_text reference U1 (at 15.24 2.54) (layer F.SilkS)
+      (effects (font (size 1 1) (thickness 0.15)))
+    )
+    (fp_text value laser_sensor (at 15.24 -2.54) (layer F.Fab)
+      (effects (font (size 1 1) (thickness 0.15)))
+    )
+    (fp_line (start 47.83 10.15) (end 47.83 -10.16) (layer F.SilkS) (width 0.15))
+    (fp_line (start 0 10.16) (end 0 -10.16) (layer F.SilkS) (width 0.15))
+    (fp_line (start 53.34 10.16) (end 49.53 10.16) (layer F.SilkS) (width 0.15))
+    (fp_line (start 0 -10.16) (end 53.34 -10.16) (layer F.SilkS) (width 0.15))
+    (fp_line (start 49.53 10.16) (end 0 10.16) (layer F.SilkS) (width 0.15))
+    (fp_text user VCC (at 7.62 -2.54) (layer F.SilkS)
+      (effects (font (size 1 1) (thickness 0.15)))
+    )
+    (fp_text user GND (at 7.62 0) (layer F.SilkS)
+      (effects (font (size 1 1) (thickness 0.15)))
+    )
+    (fp_text user DOUT (at 7.62 2.54) (layer F.SilkS)
+      (effects (font (size 1 1) (thickness 0.15)))
+    )
+    (pad 1 thru_hole circle (at 2.54 2.54) (size 1.524 1.524) (drill 0.762) (layers *.Cu *.Mask)
+      (net 3 "Net-(E1-Pad3)"))
+    (pad 2 thru_hole circle (at 2.54 0) (size 1.524 1.524) (drill 0.762) (layers *.Cu *.Mask)
+      (net 2 "Net-(E1-Pad2)"))
+    (pad 3 thru_hole circle (at 2.54 -2.54) (size 1.524 1.524) (drill 0.762) (layers *.Cu *.Mask)
+      (net 1 "Net-(E1-Pad1)"))
+  )
   (gr_line (start 231.14 85.09) (end 229.87 85.09) (angle 90) (layer Edge.Cuts) (width 0.15))
   (gr_line (start 231.14 120.65) (end 231.14 85.09) (angle 90) (layer Edge.Cuts) (width 0.15))
@@
   (gr_line (start 153.67 85.09) (end 153.67 119.38) (angle 90) (layer Edge.Cuts) (width 0.15))
   (gr_line (start 229.87 85.09) (end 153.67 85.09) (angle 90) (layer Edge.Cuts) (width 0.15))
-  (segment (start 179.07 100.33) (end 181.13 100.33) (width 0.25) (layer F.Cu) (net 1) (status 400000))
-  (segment (start 168.18 107.3) (end 167.15 106.27) (width 0.25) (layer F.Cu) (net 1) (status 800000))
+  (segment (start 179.07 100.33) (end 181.13 100.33) (width 0.25) (layer F.Cu) (net 1))
+  (segment (start 168.18 107.3) (end 167.15 106.27) (width 0.25) (layer F.Cu) (net 1))
   (segment (start 180.4 107.3) (end 168.18 107.3) (width 0.25) (layer F.Cu) (net 1))
   (segment (start 182 105.7) (end 180.4 107.3) (width 0.25) (layer F.Cu) (net 1))
   (segment (start 182 101.2) (end 182 105.7) (width 0.25) (layer F.Cu) (net 1))
   (segment (start 181.13 100.33) (end 182 101.2) (width 0.25) (layer F.Cu) (net 1))
-  (segment (start 168.93 105.25) (end 172.75 105.25) (width 0.25) (layer F.Cu) (net 2) (status 400000))
-  (segment (start 175.13 102.87) (end 179.07 102.87) (width 0.25) (layer F.Cu) (net 2) (status 800000))
+  (segment (start 168.93 105.25) (end 172.75 105.25) (width 0.25) (layer F.Cu) (net 2))
+  (segment (start 175.13 102.87) (end 179.07 102.87) (width 0.25) (layer F.Cu) (net 2))
   (segment (start 172.75 105.25) (end 175.13 102.87) (width 0.25) (layer F.Cu) (net 2))
-  (segment (start 167.15 104.23) (end 165.43 104.23) (width 0.25) (layer B.Cu) (net 3) (status 400000))
-  (segment (start 176.29 105.41) (end 179.07 105.41) (width 0.25) (layer B.Cu) (net 3) (status 800000))
+  (segment (start 167.15 104.23) (end 165.43 104.23) (width 0.25) (layer B.Cu) (net 3))
+  (segment (start 176.29 105.41) (end 179.07 105.41) (width 0.25) (layer B.Cu) (net 3))
   (segment (start 175.7 106) (end 176.29 105.41) (width 0.25) (layer B.Cu) (net 3))
   (segment (start 172 106) (end 175.7 106) (width 0.25) (layer B.Cu) (net 3))
