File: sensorPcbs/pod_health_time_of_flight/pod_health_time_of_flight.kicad_pcb (KiCad board)
At the start: 2 copper layers, 43.2 x 52.1 mm, 6 parts, among them J1 RJ45, U1 VL6180

Commit message: added all the ferkin new ethernet shields to the sensor pcbs
Parts:
- removed J1: RJ45, Connectors:RJ45_8
- added E1: RJE71-188-1401-ND, footprints:RJE71-188-1401-ND, F.Cu at (206.0, 85.0)
Connections:
- U1 pad 3: Net-(J1-Pad3) -> scl
- U1 pad 4: Net-(J1-Pad6) -> sda
- U1 pad 5: Net-(J1-Pad1) -> vcc
- U1 pad 6: Net-(J1-Pad2) -> gnd
Routing:
- net scl: track 0.00 -> 35.0 mm
- net Net-(J1-Pad1): track 18.8 -> 0.00 mm
- net vcc: track 0.00 -> 18.1 mm
- net Net-(J1-Pad6): track 15.8 -> 0.00 mm
- net gnd: track 0.00 -> 14.7 mm
- net Net-(J1-Pad3): track 13.0 -> 0.00 mm
- net Net-(J1-Pad2): track 9.94 -> 0.00 mm
- net sda: track 0.00 -> 8.96 mm

Commit message: fixed the tof according to viks wants
Parts:
- U1: footprint vl1680_footprint:VL6180 -> vl1680_footprint:tof
Changed lines of the file:
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@@
-(kicad_pcb (version 4) (host pcbnew 4.0.6)
+(kicad_pcb (version 4) (host pcbnew 4.0.3-stable)
   (general
     (links 4)
@@
     (add_net vcc)
   )
-  (module vl1680_footprint:VL6180 (layer F.Cu)
-    (at 213.36 93.98)
-    (descr "VL6180 footprint")
-    (fp_text reference U1 (at 6.35 2.54) (layer F.SilkS)
-      (effects (font (size 1 1) (thickness 0.15)))
-    )
-    (fp_text value VL6180 (at 6.35 -1.27) (layer F.Fab)
-      (effects (font (size 1 1) (thickness 0.15)))
-    )
-    (fp_arc (start 3.81 20.32) (end 7.62 20.32) (angle 90) (layer F.SilkS) (width 0.15))
-    (fp_arc (start 3.81 20.32) (end 3.81 24.13) (angle 90) (layer F.SilkS) (width 0.15))
-    (fp_arc (start 3.81 -20.32) (end 3.81 -24.13) (angle 90) (layer F.SilkS) (width 0.15))
-    (fp_arc (start 3.81 -20.32) (end 0 -20.32) (angle 90) (layer F.SilkS) (width 0.15))
-    (fp_line (start 7.62 15.24) (end 7.62 20.32) (layer F.SilkS) (width 0.15))
-    (fp_line (start 0 15.24) (end 0 20.32) (layer F.SilkS) (width 0.15))
-    (fp_line (start 7.62 -15.24) (end 7.62 -20.32) (layer F.SilkS) (width 0.15))
-    (fp_line (start 0 -15.24) (end 0 -20.32) (layer F.SilkS) (width 0.15))
-    (fp_line (start -3.81 15.24) (end 0 15.24) (layer F.SilkS) (width 0.15))
-    (fp_line (start 11.43 15.24) (end 7.62 15.24) (layer F.SilkS) (width 0.15))
-    (fp_line (start 11.43 -15.24) (end 7.62 -15.24) (layer F.SilkS) (width 0.15))
-    (fp_line (start -3.81 -15.24) (end 0 -15.24) (layer F.SilkS) (width 0.15))
-    (fp_line (start 11.43 15.24) (end 11.43 -15.24) (layer F.SilkS) (width 0.15))
-    (fp_line (start -3.81 -15.24) (end -3.81 15.24) (layer F.SilkS) (width 0.15))
-    (fp_text user SDA (at 1.27 -1.27) (layer F.SilkS)
-      (effects (font (size 1 1) (thickness 0.15)))
-    )
-    (fp_text user SCL (at 1.27 1.27 180) (layer F.SilkS)
-      (effects (font (size 1 1) (thickness 0.15)))
-    )
-    (fp_text user GND (at 1.27 -6.35) (layer F.SilkS)
-      (effects (font (size 1 1) (thickness 0.15)))
-    )
-    (fp_text user VCC (at 1.27 -3.81) (layer F.SilkS)
-      (effects (font (size 1 1) (thickness 0.15)))
-    )
-    (fp_text user IO0 (at 1.27 3.81 180) (layer F.SilkS)
-      (effects (font (size 1 1) (thickness 0.15)))
-    )
-    (fp_text user IO1 (at 1.27 6.35 180) (layer F.SilkS)
-      (effects (font (size 1 1) (thickness 0.15)))
-    )
-    (pad 3 thru_hole circle (at -2.54 1.27) (size 1.524 1.524) (drill 0.762) (layers *.Cu *.Mask)
-      (net 5 scl))
-    (pad 4 thru_hole circle (at -2.54 -1.27) (size 1.524 1.524) (drill 0.762) (layers *.Cu *.Mask)
-      (net 8 sda))
-    (pad 5 thru_hole circle (at -2.54 -3.81) (size 1.524 1.524) (drill 0.762) (layers *.Cu *.Mask)
-      (net 3 vcc))
-    (pad 2 thru_hole circle (at -2.54 3.81) (size 1.524 1.524) (drill 0.762) (layers *.Cu *.Mask)
-      (net 1 "Net-(U1-Pad2)"))
-    (pad 1 thru_hole circle (at -2.54 6.35) (size 1.524 1.524) (drill 0.762) (layers *.Cu *.Mask)
-      (net 2 "Net-(U1-Pad1)"))
-    (pad 6 thru_hole circle (at -2.54 -6.35) (size 1.524 1.524) (drill 0.762) (layers *.Cu *.Mask)
-      (net 4 gnd))
-    (pad "" thru_hole circle (at 3.81 -20.32) (size 3.048 3.048) (drill 0.762) (layers *.Cu *.Mask))
-    (pad "" thru_hole circle (at 3.81 20.32) (size 3.048 3.048) (drill 0.762) (layers *.Cu *.Mask))
-  )
   (module Connectors:1pin (layer F.Cu)
     (at 223.52 71.12)
@@
       (net 10 "Net-(E1-Pad7)"))
   )
+  (module vl1680_footprint:tof (layer F.Cu)
+    (at 213.36 93.98)
+    (descr "VL6180 footprint")
+    (fp_text reference U1 (at 6.35 2.54) (layer F.SilkS)
+      (effects (font (size 1 1) (thickness 0.15)))
+    )
+    (fp_text value VL6180 (at 6.35 -1.27) (layer F.Fab)
+      (effects (font (size 1 1) (thickness 0.15)))
+    )
+    (fp_arc (start 3.81 20.32) (end 7.62 20.32) (angle 90) (layer F.SilkS) (width 0.15))
+    (fp_arc (start 3.81 20.32) (end 3.81 24.13) (angle 90) (layer F.SilkS) (width 0.15))
+    (fp_arc (start 3.81 -20.32) (end 3.81 -24.13) (angle 90) (layer F.SilkS) (width 0.15))
+    (fp_arc (start 3.81 -20.32) (end 0 -20.32) (angle 90) (layer F.SilkS) (width 0.15))
+    (fp_line (start 7.62 15.24) (end 7.62 20.32) (layer F.SilkS) (width 0.15))
+    (fp_line (start 0 15.24) (end 0 20.32) (layer F.SilkS) (width 0.15))
+    (fp_line (start 7.62 -15.24) (end 7.62 -20.32) (layer F.SilkS) (width 0.15))
+    (fp_line (start 0 -15.24) (end 0 -20.32) (layer F.SilkS) (width 0.15))
+    (fp_line (start -3.81 15.24) (end 0 15.24) (layer F.SilkS) (width 0.15))
+    (fp_line (start 11.43 15.24) (end 7.62 15.24) (layer F.SilkS) (width 0.15))
+    (fp_line (start 11.43 -15.24) (end 7.62 -15.24) (layer F.SilkS) (width 0.15))
+    (fp_line (start -3.81 -15.24) (end 0 -15.24) (layer F.SilkS) (width 0.15))
+    (fp_line (start 11.43 15.24) (end 11.43 -15.24) (layer F.SilkS) (width 0.15))
+    (fp_line (start -3.81 -15.24) (end -3.81 15.24) (layer F.SilkS) (width 0.15))
+    (fp_text user SDA (at 1.27 -1.27) (layer F.SilkS)
+      (effects (font (size 1 1) (thickness 0.15)))
+    )
+    (fp_text user SCL (at 1.27 1.27 180) (layer F.SilkS)
+      (effects (font (size 1 1) (thickness 0.15)))
+    )
+    (fp_text user GND (at 1.27 -6.35) (layer F.SilkS)
+      (effects (font (size 1 1) (thickness 0.15)))
+    )
+    (fp_text user VCC (at 1.27 -3.81) (layer F.SilkS)
+      (effects (font (size 1 1) (thickness 0.15)))
+    )
+    (fp_text user IO0 (at 1.27 3.81 180) (layer F.SilkS)
+      (effects (font (size 1 1) (thickness 0.15)))
+    )
+    (fp_text user IO1 (at 1.27 6.35 180) (layer F.SilkS)
+      (effects (font (size 1 1) (thickness 0.15)))
+    )
+    (pad 3 thru_hole circle (at -2.54 1.27) (size 1.524 1.524) (drill 1) (layers *.Cu *.Mask)
+      (net 5 scl))
+    (pad 4 thru_hole circle (at -2.54 -1.27) (size 1.524 1.524) (drill 1) (layers *.Cu *.Mask)
+      (net 8 sda))
+    (pad 5 thru_hole circle (at -2.54 -3.81) (size 1.524 1.524) (drill 1) (layers *.Cu *.Mask)
+      (net 3 vcc))
+    (pad 2 thru_hole circle (at -2.54 3.81) (size 1.524 1.524) (drill 1) (layers *.Cu *.Mask)
+      (net 1 "Net-(U1-Pad2)"))
+    (pad 1 thru_hole circle (at -2.54 6.35) (size 1.524 1.524) (drill 1) (layers *.Cu *.Mask)
+      (net 2 "Net-(U1-Pad1)"))
+    (pad 6 thru_hole circle (at -2.54 -6.35) (size 1.524 1.524) (drill 1) (layers *.Cu *.Mask)
+      (net 4 gnd))
+  )
   (gr_line (start 184.15 67.31) (end 184.15 68.58) (angle 90) (layer Edge.Cuts) (width 0.15))
   (gr_line (start 227.33 67.31) (end 184.15 67.31) (angle 90) (layer Edge.Cuts) (width 0.15))
@@
   (gr_line (start 184.15 119.38) (end 184.15 68.58) (angle 90) (layer Edge.Cuts) (width 0.15))
   (gr_line (start 226.06 119.38) (end 184.15 119.38) (angle 90) (layer Edge.Cuts) (width 0.15))
-  (segment (start 200.55 96.67) (end 200.55 98.05) (width 0.25) (layer B.Cu) (net 3) (status 400000))
-  (segment (start 208.5 92.49) (end 210.82 90.17) (width 0.25) (layer B.Cu) (net 3) (status 800000))
+  (segment (start 200.55 96.67) (end 200.55 98.05) (width 0.25) (layer B.Cu) (net 3))
+  (segment (start 208.5 92.49) (end 210.82 90.17) (width 0.25) (layer B.Cu) (net 3))
   (segment (start 208.5 96.5) (end 208.5 92.49) (width 0.25) (layer B.Cu) (net 3))
   (segment (start 206 99) (end 208.5 96.5) (width 0.25) (layer B.Cu) (net 3))
   (segment (start 201.5 99) (end 206 99) (width 0.25) (layer B.Cu) (net 3))
   (segment (start 200.55 98.05) (end 201.5 99) (width 0.25) (layer B.Cu) (net 3))
-  (segment (start 202.33 95.65) (end 205.35 95.65) (width 0.25) (layer B.Cu) (net 4) (status 400000))
-  (segment (start 208.37 87.63) (end 210.82 87.63) (width 0.25) (layer B.Cu) (net 4) (status 800000))
+  (segment (start 202.33 95.65) (end 205.35 95.65) (width 0.25) (layer B.Cu) (net 4))
+  (segment (start 208.37 87.63) (end 210.82 87.63) (width 0.25) (layer B.Cu) (net 4))
   (segment (start 207.5 88.5) (end 208.37 87.63) (width 0.25) (layer B.Cu) (net 4))
   (segment (start 207.5 93.5) (end 207.5 88.5) (width 0.25) (layer B.Cu) (net 4))
   (segment (start 205.35 95.65) (end 207.5 93.5) (width 0.25) (layer B.Cu) (net 4))
-  (segment (start 200.55 94.63) (end 198.87 94.63) (width 0.25) (layer B.Cu) (net 5) (status 400000))
-  (segment (start 213.25 95.25) (end 210.82 95.25) (width 0.25) (layer B.Cu) (net 5) (status 800000))
+  (segment (start 200.55 94.63) (end 198.87 94.63) (width 0.25) (layer B.Cu) (net 5))
+  (segment (start 213.25 95.25) (end 210.82 95.25) (width 0.25) (layer B.Cu) (net 5))
   (segment (start 214.5 96.5) (end 213.25 95.25) (width 0.25) (layer B.Cu) (net 5))
   (segment (start 214.5 101) (end 214.5 96.5) (width 0.25) (layer B.Cu) (net 5))
@@
   (segment (start 198 95.5) (end 198 100.5) (width 0.25) (layer B.Cu) (net 5))
   (segment (start 198.87 94.63) (end 198 95.5) (width 0.25) (layer B.Cu) (net 5))
-  (segment (start 202.33 91.57) (end 206.07 91.57) (width 0.25) (layer F.Cu) (net 8) (status 400000))
-  (segment (start 207.21 92.71) (end 210.82 92.71) (width 0.25) (layer F.Cu) (net 8) (status 800000))
+  (segment (start 202.33 91.57) (end 206.07 91.57) (width 0.25) (layer F.Cu) (net 8))
+  (segment (start 207.21 92.71) (end 210.82 92.71) (width 0.25) (layer F.Cu) (net 8))
   (segment (start 206.07 91.57) (end 207.21 92.71) (width 0.25) (layer F.Cu) (net 8))
 )
